Commit message: update wrist joint type for adam_standard

File: adam_standard/adam_standard.urdf (robot description, URDF)
Before this commit: robot adam_standard, 29 links, 28 joints
Joints:
- joint wristPitch_Left: type fixed -> revolute
- joint wristPitch_Right: type fixed -> revolute
- joint wristYaw_Left: type fixed -> revolute
- joint wristYaw_Right: type fixed -> revolute
