Commit message: modif hand stl to dae for adam_sp urdf

File: adam_sp/adam_sp.urdf (robot description, URDF)
Before this commit: robot adam_sp, 55 links, 54 joints
Links:
- link L_index_distal: geometry collision mesh filename=meshes/L_index_distal.dae; visual mesh filename=meshes/L_index_distal.dae
- link L_index_proximal: geometry collision mesh filename=meshes/L_index_proximal.dae; visual mesh filename=meshes/L_index_proximal.dae
- link L_middle_distal: geometry collision mesh filename=meshes/L_middle_distal.dae; visual mesh filename=meshes/L_middle_distal.dae
- link L_middle_proximal: geometry collision mesh filename=meshes/L_middle_proximal.dae; visual mesh filename=meshes/L_middle_proximal.dae
- link L_pinky_distal: geometry collision mesh filename=meshes/L_pinky_distal.dae; visual mesh filename=meshes/L_pinky_distal.dae
- link L_pinky_proximal: geometry collision mesh filename=meshes/L_pinky_proximal.dae; visual mesh filename=meshes/L_pinky_proximal.dae
- link L_ring_distal: geometry collision mesh filename=meshes/L_ring_distal.dae; visual mesh filename=meshes/L_ring_distal.dae
- link L_ring_proximal: geometry collision mesh filename=meshes/L_ring_proximal.dae; visual mesh filename=meshes/L_ring_proximal.dae
- link L_thumb_distal: geometry collision mesh filename=meshes/L_thumb_distal.dae; visual mesh filename=meshes/L_thumb_distal.dae
- link L_thumb_intermediate: geometry collision mesh filename=meshes/L_thumb_intermediate.dae; visual mesh filename=meshes/L_thumb_intermediate.dae
- link L_thumb_proximal: geometry collision mesh filename=meshes/L_thumb_proximal.dae; visual mesh filename=meshes/L_thumb_proximal.dae
- link L_thumb_proximal_base: geometry collision mesh filename=meshes/L_thumb_proximal_base.dae; visual mesh filename=meshes/L_thumb_proximal_base.dae
- link R_index_distal: geometry collision mesh filename=meshes/R_index_distal.dae; visual mesh filename=meshes/R_index_distal.dae
- link R_index_proximal: geometry collision mesh filename=meshes/R_index_proximal.dae; visual mesh filename=meshes/R_index_proximal.dae
- link R_middle_distal: geometry collision mesh filename=meshes/R_middle_distal.dae; visual mesh filename=meshes/R_middle_distal.dae
- link R_middle_proximal: geometry collision mesh filename=meshes/R_middle_proximal.dae; visual mesh filename=meshes/R_middle_proximal.dae
- link R_pinky_distal: geometry collision mesh filename=meshes/R_pinky_distal.dae; visual mesh filename=meshes/R_pinky_distal.dae
- link R_pinky_proximal: geometry collision mesh filename=meshes/R_pinky_proximal.dae; visual mesh filename=meshes/R_pinky_proximal.dae
- link R_ring_distal: geometry collision mesh filename=meshes/R_ring_distal.dae; visual mesh filename=meshes/R_ring_distal.dae
- link R_ring_proximal: geometry collision mesh filename=meshes/R_ring_proximal.dae; visual mesh filename=meshes/R_ring_proximal.dae
- link R_thumb_distal: geometry collision mesh filename=meshes/R_thumb_distal.dae; visual mesh filename=meshes/R_thumb_distal.dae
- link R_thumb_intermediate: geometry collision mesh filename=meshes/R_thumb_intermediate.dae; visual mesh filename=meshes/R_thumb_intermediate.dae
- link R_thumb_proximal: geometry collision mesh filename=meshes/R_thumb_proximal.dae; visual mesh filename=meshes/R_thumb_proximal.dae
- link R_thumb_proximal_base: geometry collision mesh filename=meshes/R_thumb_proximal_base.dae; visual mesh filename=meshes/R_thumb_proximal_base.dae
- link wristRollLeft: geometry collision mesh filename=meshes/wristRollLeft.dae; visual mesh filename=meshes/wristRollLeft.dae
- link wristRollRight: geometry collision mesh filename=meshes/wristRollRight.dae; visual mesh filename=meshes/wristRollRight.dae
