Commit message: u

File: adam_sp/adam_sp.urdf (robot description, URDF)
Before this commit: robot adam_sp, 55 links, 54 joints
Links:
- removed link imu_link
- link L_index_distal: mass 0.009059 -> 0.00778075127730215; geometry collision mesh filename=meshes/L_index_distal.STL; visual mesh filename=meshes/L_index_distal.STL
- link L_index_proximal: mass 0.014541 -> 0.0095191609124441; geometry collision mesh filename=meshes/L_index_proximal.STL; visual mesh filename=meshes/L_index_proximal.STL
- link L_middle_distal: mass 0.009059 -> 0.00778075207653358; geometry collision mesh filename=meshes/L_middle_distal.STL; visual mesh filename=meshes/L_middle_distal.STL
- link L_middle_proximal: mass 0.013131 -> 0.00951915754527393; geometry collision mesh filename=meshes/L_middle_proximal.STL; visual mesh filename=meshes/L_middle_proximal.STL
- link L_pinky_distal: mass 0.006939 -> 0.00598769826987745; geometry collision mesh filename=meshes/L_pinky_distal.STL; visual mesh filename=meshes/L_pinky_distal.STL
- link L_pinky_proximal: mass 0.013131 -> 0.00951915508482644; geometry collision mesh filename=meshes/L_pinky_proximal.STL; visual mesh filename=meshes/L_pinky_proximal.STL
- link L_ring_distal: mass 0.009059 -> 0.00778076129148193; geometry collision mesh filename=meshes/L_ring_distal.STL; visual mesh filename=meshes/L_ring_distal.STL
- link L_ring_proximal: mass 0.014541 -> 0.00951915061644606; geometry collision mesh filename=meshes/L_ring_proximal.STL; visual mesh filename=meshes/L_ring_proximal.STL
- link L_thumb_distal: mass 0.010437 -> 0.00929919523909398; geometry collision mesh filename=meshes/L_thumb_distal.STL; visual mesh filename=meshes/L_thumb_distal.STL
- link L_thumb_intermediate: mass 0.015383 -> 0.010692760480567; geometry collision mesh filename=meshes/L_thumb_intermediate.STL; visual mesh filename=meshes/L_thumb_intermediate.STL
- link L_thumb_proximal: mass 0.061584 -> 0.0264126544762834; geometry collision mesh filename=meshes/L_thumb_proximal.STL; visual mesh filename=meshes/L_thumb_proximal.STL
- link L_thumb_proximal_base: mass 0.0089319 -> 0.00574531091218956; geometry collision mesh filename=meshes/L_thumb_proximal_base.STL; visual mesh filename=meshes/L_thumb_proximal_base.STL
- link R_index_distal: mass 0.009059 -> 0.007780916719648; geometry collision mesh filename=meshes/R_index_distal.STL; visual mesh filename=meshes/R_index_distal.STL
- link R_index_proximal: mass 0.014541 -> 0.00951915775379086; geometry collision mesh filename=meshes/R_index_proximal.STL; visual mesh filename=meshes/R_index_proximal.STL
- link R_middle_distal: mass 0.009059 -> 0.00778091288583433; geometry collision mesh filename=meshes/R_middle_distal.STL; visual mesh filename=meshes/R_middle_distal.STL
- link R_middle_proximal: mass 0.013131 -> 0.00951915853498458; geometry collision mesh filename=meshes/R_middle_proximal.STL; visual mesh filename=meshes/R_middle_proximal.STL
- link R_pinky_distal: mass 0.006939 -> 0.0059874955616141; geometry collision mesh filename=meshes/R_pinky_distal.STL; visual mesh filename=meshes/R_pinky_distal.STL
- link R_pinky_proximal: mass 0.013131 -> 0.00951915301881843; geometry collision mesh filename=meshes/R_pinky_proximal.STL; visual mesh filename=meshes/R_pinky_proximal.STL
- link R_ring_distal: mass 0.009059 -> 0.00778091436084645; geometry collision mesh filename=meshes/R_ring_distal.STL; visual mesh filename=meshes/R_ring_distal.STL
- link R_ring_proximal: mass 0.014541 -> 0.00951915034399878; geometry collision mesh filename=meshes/R_ring_proximal.STL; visual mesh filename=meshes/R_ring_proximal.STL
- link R_thumb_distal: mass 0.010437 -> 0.00930094539471516; geometry collision mesh filename=meshes/R_thumb_distal.STL; visual mesh filename=meshes/R_thumb_distal.STL
- link R_thumb_intermediate: mass 0.015383 -> 0.0106927627467546; geometry collision mesh filename=meshes/R_thumb_intermediate.STL; visual mesh filename=meshes/R_thumb_intermediate.STL
- link R_thumb_proximal: mass 0.061584 -> 0.0264126768516325; geometry collision mesh filename=meshes/R_thumb_proximal.STL; visual mesh filename=meshes/R_thumb_proximal.STL
- link R_thumb_proximal_base: mass 0.0089319 -> 0.00574530987842469; geometry collision mesh filename=meshes/R_thumb_proximal_base.STL; visual mesh filename=meshes/R_thumb_proximal_base.STL
- link anklePitchLeft: mass 0.03014230 -> 0.00668343610831866; geometry collision mesh filename=meshes/anklePitchLeft.STL; visual mesh filename=meshes/anklePitchLeft.STL
- link anklePitchRight: mass 0.03014230 -> 0.00668343610831867; geometry collision mesh filename=meshes/anklePitchRight.STL; visual mesh filename=meshes/anklePitchRight.STL
- link elbowLeft: mass 0.85400000 -> 0.0732555409052303; geometry collision mesh filename=meshes/elbowLeft.STL; visual mesh filename=meshes/elbowLeft.STL
- link elbowRight: mass 0.85400000 -> 0.0732555404902823; geometry collision mesh filename=meshes/elbowRight.STL; visual mesh filename=meshes/elbowRight.STL
- link hipPitchLeft: mass 2.23379987 -> 0.692207569187135; geometry collision mesh filename=meshes/hipPitchLeft.STL; visual mesh filename=meshes/hipPitchLeft.STL
- link hipPitchRight: mass 2.23477271 -> 0.692205170637013; geometry collision mesh filename=meshes/hipPitchRight.STL; visual mesh filename=meshes/hipPitchRight.STL
- link hipRollLeft: mass 1.35107789 -> 0.401082499974616; geometry collision mesh filename=meshes/hipRollLeft.STL; visual mesh filename=meshes/hipRollLeft.STL
- link hipRollRight: mass 1.35169943 -> 0.40108507388712; geometry collision mesh filename=meshes/hipRollRight.STL; visual mesh filename=meshes/hipRollRight.STL
- link pelvis: mass 10.35646604 -> 3.54360274725497; geometry collision mesh filename=meshes/pelvis.STL; visual mesh filename=meshes/pelvis.STL
- link shinLeft: mass 2.25363003 -> 0.645968928229465; geometry collision mesh filename=meshes/shinLeft.STL; visual mesh filename=meshes/shinLeft.STL
- link shinRight: mass 2.25459286 -> 0.644290991404595; geometry collision mesh filename=meshes/shinRight.STL; visual mesh filename=meshes/shinRight.STL
- link shoulderPitchLeft: mass 0.20310000 -> 0.0720079227497436; geometry collision mesh filename=meshes/shoulderPitchLeft.STL; visual mesh filename=meshes/shoulderPitchLeft.STL
- link shoulderPitchRight: mass 0.20310000 -> 0.0720080684790082; geometry collision mesh filename=meshes/shoulderPitchRight.STL; visual mesh filename=meshes/shoulderPitchRight.STL
- link shoulderRollLeft: mass 0.72480000 -> 0.220148586716196; geometry collision mesh filename=meshes/shoulderRollLeft.STL; visual mesh filename=meshes/shoulderRollLeft.STL
- link shoulderRollRight: mass 0.72480000 -> 0.220149768456595; geometry collision mesh filename=meshes/shoulderRollRight.STL; visual mesh filename=meshes/shoulderRollRight.STL
- link shoulderYawLeft: mass 0.69630000 -> 16.7008523306088; geometry collision mesh filename=meshes/shoulderYawLeft.STL; visual mesh filename=meshes/shoulderYawLeft.STL
- link shoulderYawRight: mass 0.69630000 -> 16.7008523306088; geometry collision mesh filename=meshes/shoulderYawRight.STL; visual mesh filename=meshes/shoulderYawRight.STL
- link thighLeft: mass 6.43432838 -> 2.02546553651926; geometry collision mesh filename=meshes/thighLeft.STL; visual mesh filename=meshes/thighLeft.STL
- link thighRight: mass 6.43084152 -> 2.02467766041122; geometry collision mesh filename=meshes/thighRight.STL; visual mesh filename=meshes/thighRight.STL
- link toeLeft: mass 0.63479601 -> 0.400347849670894; geometry collision mesh filename=meshes/toeLeft.STL; visual mesh filename=meshes/toeLeft.STL
- link toeRight: mass 0.63480789 -> 0.402799762004053; geometry collision mesh filename=meshes/toeRight.STL; visual mesh filename=meshes/toeRight.STL
- link torso: mass 12.89652496 -> 1.75951184587366; geometry collision mesh filename=meshes/torso.STL; visual mesh filename=meshes/torso.STL
- link waistPitch: mass 0.56353776 -> 0.188254684395963; geometry collision mesh filename=meshes/waistPitch.STL; visual mesh filename=meshes/waistPitch.STL
- link waistRoll: mass 2.36268465 -> 0.674091084130766; geometry collision mesh filename=meshes/waistRoll.STL; visual mesh filename=meshes/waistRoll.STL
- link wristPitchLeft: mass 0.11963454 -> 0.0380100074372544; geometry collision mesh filename=meshes/wristPitchLeft.STL; visual mesh filename=meshes/wristPitchLeft.STL
- link wristPitchRight: mass 0.11963454 -> 0.0405153415237362; geometry collision mesh filename=meshes/wristPitchRight.STL; visual mesh filename=meshes/wristPitchRight.STL
- link wristRollLeft: mass 0.3575 -> 0.184675835731943; geometry collision mesh filename=meshes/wristRollLeft.STL; visual mesh filename=meshes/wristRollLeft.STL
- link wristRollRight: mass 0.35816 -> 0.184672295298046; geometry collision mesh filename=meshes/wristRollRight.STL; visual mesh filename=meshes/wristRollRight.STL
- link wristYawLeft: mass 0.95587869 -> 0.366169801573267; geometry collision mesh filename=meshes/wristYawLeft.STL; visual mesh filename=meshes/wristYawLeft.STL
- link wristYawRight: mass 0.95587832 -> 0.380961652216889; geometry collision mesh filename=meshes/wristYawRight.STL; visual mesh filename=meshes/wristYawRight.STL
Joints:
- removed joint Lindex_distal
- removed joint Lindex_proximal
- removed joint Lmiddle_distal
- removed joint Lmiddle_proximal
- removed joint Lpinky_distal
- removed joint Lpinky_proximal
- removed joint Lring_distal
- removed joint Lring_proximal
- removed joint Lthumb_distal
- removed joint Lthumb_intermediate
- removed joint Lthumb_proximal
- removed joint Lthumb_proximal_base
- removed joint Rindex_distal
- removed joint Rindex_proximal
- removed joint Rmiddle_distal
- removed joint Rmiddle_proximal
- removed joint Rpinky_distal
- removed joint Rpinky_proximal
- removed joint Rring_distal
- removed joint Rring_proximal
- removed joint Rthumb_distal
- removed joint Rthumb_intermediate
- removed joint Rthumb_proximal
- removed joint Rthumb_proximal_base
- removed joint imu_joint
- added joint L_index_DIP_joint: type continuous, parent L_index_proximal, child L_index_distal, origin xyz=0 -0.00111268989731944 -0.0319806491677784 rpy=0 0 0, axis -1 0 0
- added joint L_index_MCP_joint: type continuous, parent wristRollLeft, child L_index_proximal, origin xyz=0.0269420472022218 0.00950000000154763 -0.114975331627829 rpy=0 -0.0523598774782631 0, axis -1 0 0
- added joint L_middle_DIP_joint: type continuous, parent L_middle_proximal, child L_middle_distal, origin xyz=0 -0.00293735370583337 -0.0318649015879072 rpy=0 0 0, axis -1 0 0
- added joint L_middle_MCP_joint: type continuous, parent wristRollLeft, child L_middle_proximal, origin xyz=0.00799999998838565 0.0144999999999475 -0.128000000000728 rpy=0 0 0, axis -1 0 0
- added joint L_pinky_DIP_joint: type continuous, parent L_pinky_proximal, child L_pinky_distal, origin xyz=0 -0.00111268989776986 -0.0319806491677628 rpy=0 0 0, axis -1 0 0
- added joint L_pinky_MCP_joint: type continuous, parent wristRollLeft, child L_pinky_proximal, origin xyz=-0.0301936481908677 0.00449999999694281 -0.11286583072711 rpy=0 0.12217304772112 0, axis -1 0 0
- added joint L_ring_DIP_joint: type continuous, parent L_ring_proximal, child L_ring_distal, origin xyz=0 -0.00111268989759014 -0.0319806491677691 rpy=0 0 0, axis -1 0 0
- added joint L_ring_MCP_joint: type continuous, parent wristRollLeft, child L_ring_proximal, origin xyz=-0.0109420472229284 0.00949999999845705 -0.119975331624717 rpy=0 0.052359877641387 0, axis -1 0 0
- added joint L_thumb_DIP_joint: type continuous, parent L_thumb_intermediate, child L_thumb_distal, origin xyz=0.0164679343341741 0 -0.0154614727230483 rpy=0 0 0, axis 0 1 0
- added joint L_thumb_MCP_joint1: type continuous, parent wristRollLeft, child L_thumb_proximal_base, origin xyz=0.0244999999969742 -0.0099999999982788 -0.0470000000019433 rpy=0 0 0, axis 0 0 1
- added joint L_thumb_MCP_joint2: type continuous, parent L_thumb_proximal_base, child L_thumb_proximal, origin xyz=0.011954002456522 -0.00104967865057148 0 rpy=0 0 -0.0875851578962738, axis 0 1 0
- added joint L_thumb_PIP_joint: type continuous, parent L_thumb_proximal, child L_thumb_intermediate, origin xyz=0.0442885641132063 0 -0.0376632856876562 rpy=0 0 0, axis 0 1 0
- added joint R_index_DIP_joint: type continuous, parent R_index_proximal, child R_index_distal, origin xyz=0 0.00111268989722751 -0.0319806491677816 rpy=0 0 0, axis 1 0 0
- added joint R_index_MCP_joint: type continuous, parent wristRollRight, child R_index_proximal, origin xyz=0.0269420472120735 -0.00950000000009146 -0.114975331625641 rpy=0 -0.0523598775568891 0, axis 1 0 0
- added joint R_middle_DIP_joint: type continuous, parent R_middle_proximal, child R_middle_distal, origin xyz=0 0.00293735370559906 -0.0318649015879289 rpy=0 0 0, axis 1 0 0
- added joint R_middle_MCP_joint: type continuous, parent wristRollRight, child R_middle_proximal, origin xyz=0.00799999999968861 -0.0145000000002054 -0.127999999999992 rpy=0 0 0, axis 1 0 0
- added joint R_pinky_DIP_joint: type continuous, parent R_pinky_proximal, child R_pinky_distal, origin xyz=0 0.00111268989720342 -0.0319806491677825 rpy=0 0 0, axis 1 0 0
- added joint R_pinky_MCP_joint: type continuous, parent wristRollRight, child R_pinky_proximal, origin xyz=-0.0301936481816091 -0.00450000000035261 -0.112865830729451 rpy=0 0.122173047642494 0, axis 1 0 0
- added joint R_ring_DIP_joint: type continuous, parent R_ring_proximal, child R_ring_distal, origin xyz=0 0.00111268989721214 -0.0319806491677822 rpy=0 0 0, axis 1 0 0
- added joint R_ring_MCP_joint: type continuous, parent wristRollRight, child R_ring_proximal, origin xyz=-0.0109420472126836 -0.00950000000027432 -0.119975331625507 rpy=0 0.0523598775627611 0, axis 1 0 0
- added joint R_thumb_DIP_joint: type continuous, parent R_thumb_intermediate, child R_thumb_distal, origin xyz=0.0164679343353944 0 -0.0154614727217485 rpy=0 0 0, axis 0 1 0
- added joint R_thumb_MCP_joint1: type continuous, parent wristRollRight, child R_thumb_proximal_base, origin xyz=0.0244999999998152 0.0100000000000263 -0.0470000000000906 rpy=0 0 0, axis 0 0 -1
- added joint R_thumb_MCP_joint2: type continuous, parent R_thumb_proximal_base, child R_thumb_proximal, origin xyz=0.0119540024564323 0.00104967865159283 0 rpy=0 0 0.0875851579817108, axis 0 1 0
- added joint R_thumb_PIP_joint: type continuous, parent R_thumb_proximal, child R_thumb_intermediate, origin xyz=0.044288564116179 0 -0.0376632856841606 rpy=0 0 0, axis 0 1 0
- joint anklePitch_Left: axis 0 1 0 -> 0 0.999999999999993 0; limit lower=-1.0 upper=0.35 effort=40.0 velocity=20.0 -> (none); origin xyz=0 0 -0.37 rpy=0 0 0 -> xyz=0 0 -0.36999999999995 rpy=0 0 0; type revolute -> continuous
- joint anklePitch_Right: axis 0 1 0 -> 0 -0.999999999999932 0; limit lower=-1.0 upper=0.35 effort=40.0 velocity=20.0 -> (none); origin xyz=0 0 -0.37 rpy=0 0 0 -> xyz=0 0 -0.369999999999911 rpy=0 0 0; type revolute -> continuous
- joint ankleRoll_Left: axis 1 0 0 -> -0.999999999999984 0 0; limit lower=-0.3491 upper=0.3491 effort=12.0 velocity=20.0 -> (none); type revolute -> continuous
- joint ankleRoll_Right: axis 1 0 0 -> 0.999999999999795 0 0; limit lower=-0.3491 upper=0.3491 effort=12.0 velocity=20.0 -> (none); type revolute -> continuous
- joint elbow_Left: axis 0 1 0 -> 0 -1 0; limit lower=-2.0 upper=0.0 effort=30.0 velocity=8.0 -> (none); origin xyz=0 -0.0285 -0.20415 rpy=0 0 0 -> xyz=0 -0.0285000000009982 -0.182950000001738 rpy=0 0 0; type revolute -> continuous
- joint elbow_Right: limit lower=-2.0 upper=0.0 effort=30.0 velocity=8.0 -> (none); origin xyz=0 0.0285 -0.20415 rpy=0 0 0 -> xyz=0 0.0284999999998828 -0.182950000001922 rpy=0 0 0; type revolute -> continuous
- joint hipPitch_Left: axis 0 1 0 -> 0 -1 0; limit lower=-2.164 upper=2.164 effort=230.0 velocity=15.0 -> (none); origin xyz=0 0.096192 -0.033241 rpy=-0.61087 0 0 -> xyz=0 0.0961924921295064 -0.0332411879418571 rpy=-0.610865238197473 0 0; type revolute -> continuous
- joint hipPitch_Right: axis 0 1 0 -> 0 -1 0; limit lower=-2.164 upper=2.164 effort=230.0 velocity=15.0 -> (none); origin xyz=0 -0.096192 -0.033241 rpy=0.61087 0 0 -> xyz=0 -0.0961924781696877 -0.0332412045786055 rpy=0.610865238197555 0 0; type revolute -> continuous
- joint hipRoll_Left: axis 1 0 0 -> -0.999999999999984 0 0; limit lower=-0.733 upper=1.605 effort=160.0 velocity=8.0 -> (none); origin xyz=-0.0255 0.069 0 rpy=0.61087 0 0 -> xyz=-0.0254999999999983 0.0690000000000026 0 rpy=0.610865238197473 0 0; type revolute -> continuous
- joint hipRoll_Right: axis 1 0 0 -> 0.999999999999795 0 0; limit lower=-1.605 upper=0.733 effort=160.0 velocity=8.0 -> (none); origin xyz=-0.0255 -0.069 0 rpy=-0.61087 0 0 -> xyz=-0.0254999999999981 -0.0689999999999357 0 rpy=-0.610865238197555 0 0; type revolute -> continuous
- joint hipYaw_Left: axis 0 0 1 -> 0 0 0.999999999999991; limit lower=-0.785 upper=0.785 effort=105 velocity=8.0 -> (none); origin xyz=0.044 0 -0.0525 rpy=0 0 0 -> xyz=0.0440000071360198 0 -0.0524999940193389 rpy=0 0 0; type revolute -> continuous
- joint hipYaw_Right: axis 0 0 1 -> 0 0 -0.999999999999862; limit lower=-0.785 upper=0.785 effort=105 velocity=8.0 -> (none); origin xyz=0.044 0 -0.0525 rpy=0 0 0 -> xyz=0.0439999724402559 0 -0.0525000230976866 rpy=0 0 0; type revolute -> continuous
- joint kneePitch_Left: axis 0 1 0 -> 0 0.999999999999993 0; limit lower=0.052 upper=2.391 effort=230.0 velocity=15.0 -> (none); origin xyz=0 -0.0355 -0.369 rpy=0 0 0 -> xyz=0 -0.0354999999998497 -0.369000000000099 rpy=0 0 0; type revolute -> continuous
- joint kneePitch_Right: axis 0 1 0 -> 0 0.999999999999932 0; limit lower=0.052 upper=2.391 effort=230.0 velocity=15.0 -> (none); origin xyz=0 0.0355 -0.369 rpy=0 0 0 -> xyz=0 0.0354999999997395 -0.368999999999986 rpy=0 0 0; type revolute -> continuous
- joint shoulderPitch_Left: limit lower=-3.560 upper=1.989 effort=65.0 velocity=8.0 -> (none); origin xyz=0 0.16011 0.25742 rpy=0.34907 0 0 -> xyz=0 0.165093970689425 0.259229560594865 rpy=0.349065850393456 0 0; type revolute -> continuous
- joint shoulderPitch_Right: axis 0 1 0 -> 0 -1 0; limit lower=-3.560 upper=1.989 effort=65.0 velocity=8.0 -> (none); origin xyz=0 -0.16011 0.25742 rpy=-0.34907 0 0 -> xyz=0 -0.165093970689321 0.259229560595242 rpy=-0.349065850398898 0 0; type revolute -> continuous
- joint shoulderRoll_Left: limit lower=-0.575 upper=2.74 effort=65.0 velocity=8.0 -> (none); origin xyz=0.0335 0.0435 0 rpy=-0.34907 0 0 -> xyz=0.036199999996826 0.0434999999975074 0 rpy=-0.349065850393456 0 0; type revolute -> continuous
- joint shoulderRoll_Right: limit lower=-2.74 upper=0.575 effort=65.0 velocity=8.0 -> (none); origin xyz=0.0335 -0.0435 0 rpy=0.34907 0 0 -> xyz=0.036199999639011 -0.0435000000171988 0 rpy=0.349065850398898 0 0; type revolute -> continuous
- joint shoulderYaw_Left: limit lower=-1.6 upper=1.6 effort=65.0 velocity=8.0 -> (none); origin xyz=-0.0335 0.034 -0.0585 rpy=0 0 0 -> xyz=-0.0361999999622004 0.0340000000110588 -0.0796999999903454 rpy=0 0 0; type revolute -> continuous
- joint shoulderYaw_Right: limit lower=-1.6 upper=1.6 effort=65.0 velocity=8.0 -> (none); origin xyz=-0.0335 -0.034 -0.0585 rpy=0 0 0 -> xyz=-0.0361999996389017 -0.0339999999996759 -0.0797000000498751 rpy=0 0 0; type revolute -> continuous
- joint waistPitch: axis 0 1 0 -> 0 -1 0; limit lower=-0.785 upper=1.308 effort=110 velocity=8.0 -> (none); type revolute -> continuous
- joint waistRoll: limit lower=-0.226 upper=0.226 effort=110 velocity=8.0 -> (none); origin xyz=0 0 0.044 rpy=0 0 0 -> xyz=0 0 0.0440000000007929 rpy=0 0 0; type revolute -> continuous
- joint waistYaw: axis 0 0 1 -> 0 0 -1; limit lower=-0.78 upper=0.78 effort=110 velocity=8.0 -> (none); origin xyz=0 0.0005 0.053 rpy=0 0 0 -> xyz=0 0.000500000000007081 0.05299999999999 rpy=0 0 0; type revolute -> continuous
- joint wristPitch_Left: limit lower=-0.907 upper=0.907 effort=6.4 velocity=4.9218 -> (none); origin xyz=0 0 -0.2017 rpy=0 0 0 -> xyz=0 0 -0.201699999999994 rpy=0 0 0; type revolute -> continuous
- joint wristPitch_Right: limit lower=-0.907 upper=0.907 effort=6.4 velocity=4.9218 -> (none); origin xyz=0 0 -0.201699999719004 rpy=0 0 0 -> xyz=0 0 -0.201699999999861 rpy=0 0 0; type revolute -> continuous
- joint wristRoll_Left: limit lower=-0.907 upper=0.907 effort=6.4 velocity=4.9218 -> (none); type revolute -> continuous
- joint wristRoll_Right: axis 1 0 0 -> -1 0 0; limit lower=-0.907 upper=0.907 effort=6.4 velocity=4.9218 -> (none); type revolute -> continuous
- joint wristYaw_Left: limit lower=-2.617 upper=2.617 effort=6.4 velocity=4.9218 -> (none); origin xyz=-0.025 0.0285 -0.0729 rpy=0 0 0 -> xyz=-0.0250000000083053 0.028499999997574 -0.0728999999980683 rpy=0 0 0; type revolute -> continuous
- joint wristYaw_Right: limit lower=-2.617 upper=2.617 effort=6.4 velocity=4.9218 -> (none); origin xyz=-0.025 -0.0285 -0.0729 rpy=0 0 0 -> xyz=-0.0249999999999065 -0.0285000000002922 -0.0728999999999894 rpy=0 0 0; type revolute -> continuous

Commit message: update link name

File: adam_sp/adam_sp.urdf (robot description, URDF)
Before this commit: robot adam-sp-pvt2, 54 links, 53 joints
Links:
- removed link waistPitch
- removed link waistRoll
- added link waistPitch_link, mass 0.188254684395963; collision mesh filename=meshes/waistPitch.STL; visual mesh filename=meshes/waistPitch.STL
- added link waistRoll_link, mass 0.674091084130766; collision mesh filename=meshes/waistRoll.STL; visual mesh filename=meshes/waistRoll.STL

File: adam_u/adam_u.urdf (robot description, URDF)
Before this commit: robot adam_u, 44 links, 43 joints
Links:
- removed link neckPitch
- removed link neckYaw
- removed link waistPitch
- removed link waistRoll
- added link neckPitch_link, mass 0.99740875; collision mesh filename=meshes_stl_0.25/neckPitch.STL; visual mesh filename=meshes_dae/neckPitch.dae
- added link neckYaw_link, mass 0.41242410; collision mesh filename=meshes_stl_0.25/neckYaw.STL; visual mesh filename=meshes_dae/neckYaw.dae
- added link waistPitch_link, mass 0.56353776; collision mesh filename=meshes_stl_0.25/waistPitch.STL; visual mesh filename=meshes_dae/waistPitch.dae
- added link waistRoll_link, mass 2.36268465; collision mesh filename=meshes_stl_0.25/waistRoll.STL; visual mesh filename=meshes_dae/waistRoll.dae
