Commit message: update adam_sp mass inertia

File: adam_sp/adam_sp.urdf (robot description, URDF)
Before this commit: robot adam_sp, 54 links, 53 joints
Links:
- link L_index_distal: mass 0.00778075127730215 -> 0.00905901
- link L_index_proximal: mass 0.0095191609124441 -> 0.01454111
- link L_middle_distal: mass 0.00778075207653358 -> 0.00905901
- link L_middle_proximal: mass 0.00951915754527393 -> 0.01313099
- link L_pinky_distal: mass 0.00598769826987745 -> 0.00693901
- link L_pinky_proximal: mass 0.00951915508482644 -> 0.01313099
- link L_ring_distal: mass 0.00778076129148193 -> 0.00905901
- link L_ring_proximal: mass 0.00951915061644606 -> 0.01454111
- link L_thumb_distal: mass 0.00929919523909398 -> 0.01043740
- link L_thumb_intermediate: mass 0.010692760480567 -> 0.01538337
- link L_thumb_proximal: mass 0.0264126544762834 -> 0.06158427
- link L_thumb_proximal_base: mass 0.00574531091218956 -> 0.00893190
- link R_index_distal: mass 0.007780916719648 -> 0.00905901
- link R_index_proximal: mass 0.00951915775379086 -> 0.01454119
- link R_middle_distal: mass 0.00778091288583433 -> 0.00905901
- link R_middle_proximal: mass 0.00951915853498458 -> 0.01313107
- link R_pinky_distal: mass 0.0059874955616141 -> 0.00693901
- link R_pinky_proximal: mass 0.00951915301881843 -> 0.01313107
- link R_ring_distal: mass 0.00778091436084645 -> 0.00905901
- link R_ring_proximal: mass 0.00951915034399878 -> 0.01454119
- link R_thumb_distal: mass 0.00930094539471516 -> 0.01043741
- link R_thumb_intermediate: mass 0.0106927627467546 -> 0.01538338
- link R_thumb_proximal: mass 0.0264126768516325 -> 0.06158426
- link R_thumb_proximal_base: mass 0.00574530987842469 -> 0.00893190
- link anklePitchLeft: mass 0.00668343610831866 -> 0.03014230
- link anklePitchRight: mass 0.00668343610831867 -> 0.03014230
- link elbowLeft: mass 0.0732555409052303 -> 0.91770702
- link elbowRight: mass 0.0732555404902823 -> 0.91770702
- link hipPitchLeft: mass 0.692207569187135 -> 2.23379987
- link hipPitchRight: mass 0.692205170637013 -> 2.23477271
- link hipRollLeft: mass 0.401082499974616 -> 1.35107789
- link hipRollRight: mass 0.40108507388712 -> 1.35169943
- link pelvis: mass 3.54360274725497 -> 10.35646604
- link shinLeft: mass 0.645968928229465 -> 2.25363003
- link shinRight: mass 0.644290991404595 -> 2.25459286
- link shoulderPitchLeft: mass 0.0720079227497436 -> 0.21614811
- link shoulderPitchRight: mass 0.0720080684790082 -> 0.21648747
- link shoulderRollLeft: mass 0.220148586716196 -> 1.07881773
- link shoulderRollRight: mass 0.220149768456595 -> 1.08875448
- link shoulderYawLeft: mass 16.7008523306088 -> 0.90142027
- link shoulderYawRight: mass 16.7008523306088 -> 0.90139273
- link thighLeft: mass 2.02546553651926 -> 6.43432838
- link thighRight: mass 2.02467766041122 -> 6.43084152
- link toeLeft: mass 0.400347849670894 -> 0.63479601
- link toeRight: mass 0.402799762004053 -> 0.63480789
- link torso: mass 1.75951184587366 -> 13.46342537
- link waistPitch_link: mass 0.188254684395963 -> 0.56353776
- link waistRoll_link: mass 0.674091084130766 -> 2.36268465
- link wristPitchLeft: mass 0.0380100074372544 -> 0.11963454
- link wristPitchRight: mass 0.0405153415237362 -> 0.11963454
- link wristRollLeft: mass 0.184675835731943 -> 0.35749661
- link wristRollRight: mass 0.184672295298046 -> 0.35815530
- link wristYawLeft: mass 0.366169801573267 -> 0.95587869
- link wristYawRight: mass 0.380961652216889 -> 0.95587832

Commit message: update axis, add limit

File: adam_sp/adam_sp.urdf (robot description, URDF)
Before this commit: robot adam_sp, 54 links, 53 joints
Joints:
- joint L_index_DIP_joint: limit (none) -> lower=0 upper=1.6 effort=1 velocity=1; type continuous -> revolute
- joint L_index_MCP_joint: limit (none) -> lower=0 upper=1.7 effort=1 velocity=1; type continuous -> revolute
- joint L_middle_DIP_joint: limit (none) -> lower=0 upper=1.6 effort=1 velocity=1; type continuous -> revolute
- joint L_middle_MCP_joint: limit (none) -> lower=0 upper=1.7 effort=1 velocity=1; type continuous -> revolute
- joint L_pinky_DIP_joint: limit (none) -> lower=0 upper=1.6 effort=1 velocity=1; type continuous -> revolute
- joint L_pinky_MCP_joint: limit (none) -> lower=0 upper=1.7 effort=1 velocity=1; type continuous -> revolute
- joint L_ring_DIP_joint: limit (none) -> lower=0 upper=1.6 effort=1 velocity=1; type continuous -> revolute
- joint L_ring_MCP_joint: limit (none) -> lower=0 upper=1.7 effort=1 velocity=1; type continuous -> revolute
- joint L_thumb_DIP_joint: limit (none) -> lower=0 upper=1.2 effort=1 velocity=1; type continuous -> revolute
- joint L_thumb_MCP_joint1: axis 0 0 1 -> 0 0 -1; limit (none) -> lower=0 upper=1.1 effort=1 velocity=1; type continuous -> revolute
- joint L_thumb_MCP_joint2: limit (none) -> lower=0 upper=0.5 effort=1 velocity=1; type continuous -> revolute
- joint L_thumb_PIP_joint: limit (none) -> lower=0 upper=1 effort=1 velocity=1; type continuous -> revolute
- joint R_index_DIP_joint: limit (none) -> lower=0 upper=1.6 effort=1 velocity=1; type continuous -> revolute
- joint R_index_MCP_joint: limit (none) -> lower=0 upper=1.7 effort=1 velocity=1; type continuous -> revolute
- joint R_middle_DIP_joint: limit (none) -> lower=0 upper=1.6 effort=1 velocity=1; type continuous -> revolute
- joint R_middle_MCP_joint: limit (none) -> lower=0 upper=1.7 effort=1 velocity=1; type continuous -> revolute
- joint R_pinky_DIP_joint: limit (none) -> lower=0 upper=1.6 effort=1 velocity=1; type continuous -> revolute
- joint R_pinky_MCP_joint: limit (none) -> lower=0 upper=1.7 effort=1 velocity=1; type continuous -> revolute
- joint R_ring_DIP_joint: limit (none) -> lower=0 upper=1.6 effort=1 velocity=1; type continuous -> revolute
- joint R_ring_MCP_joint: limit (none) -> lower=0 upper=1.7 effort=1 velocity=1; type continuous -> revolute
- joint R_thumb_DIP_joint: limit (none) -> lower=0 upper=1.2 effort=1 velocity=1; type continuous -> revolute
- joint R_thumb_MCP_joint1: axis 0 0 -1 -> 0 0 1; limit (none) -> lower=0 upper=1.1 effort=1 velocity=1; type continuous -> revolute
- joint R_thumb_MCP_joint2: limit (none) -> lower=0 upper=0.5 effort=1 velocity=1; type continuous -> revolute
- joint R_thumb_PIP_joint: limit (none) -> lower=0 upper=1 effort=1 velocity=1; type continuous -> revolute
- joint anklePitch_Left: axis 0 0.999999999999993 0 -> 0 1 0; limit (none) -> lower=-1.0 upper=0.35 effort=40 velocity=20; type continuous -> revolute
- joint anklePitch_Right: axis 0 -0.999999999999932 0 -> 0 1 0; limit (none) -> lower=-1.0 upper=0.35 effort=40 velocity=20; type continuous -> revolute
- joint ankleRoll_Left: axis -0.999999999999984 0 0 -> 1 0 0; limit (none) -> lower=-0.3491 upper=0.3491 effort=12 velocity=20; type continuous -> revolute
- joint ankleRoll_Right: axis 0.999999999999795 0 0 -> 1 0 0; limit (none) -> lower=-0.3491 upper=0.3491 effort=12 velocity=20; type continuous -> revolute
- joint elbow_Left: axis 0 -1 0 -> 0 1 0; limit (none) -> lower=-2.496 upper=0.209 effort=30 velocity=8; type continuous -> revolute
- joint elbow_Right: limit (none) -> lower=-2.496 upper=0.209 effort=30 velocity=8; type continuous -> revolute
- joint hipPitch_Left: axis 0 -1 0 -> 0 1 0; limit (none) -> lower=-2.164 upper=2.164 effort=230 velocity=15; type continuous -> revolute
- joint hipPitch_Right: axis 0 -1 0 -> 0 1 0; limit (none) -> lower=-2.164 upper=2.164 effort=230 velocity=15; type continuous -> revolute
- joint hipRoll_Left: axis -0.999999999999984 0 0 -> 1 0 0; limit (none) -> lower=-0.733 upper=1.605 effort=160 velocity=8; type continuous -> revolute
- joint hipRoll_Right: axis 0.999999999999795 0 0 -> 1 0 0; limit (none) -> lower=-1.605 upper=0.733 effort=160 velocity=8; type continuous -> revolute
- joint hipYaw_Left: axis 0 0 0.999999999999991 -> 0 0 1; limit (none) -> lower=-0.785 upper=0.785 effort=105 velocity=8; type continuous -> revolute
- joint hipYaw_Right: axis 0 0 -0.999999999999862 -> 0 0 1; limit (none) -> lower=-0.785 upper=0.785 effort=105 velocity=8; type continuous -> revolute
- joint kneePitch_Left: axis 0 0.999999999999993 0 -> 0 1 0; limit (none) -> lower=0.052 upper=2.391 effort=230 velocity=15; type continuous -> revolute
- joint kneePitch_Right: axis 0 0.999999999999932 0 -> 0 1 0; limit (none) -> lower=0.052 upper=2.391 effort=230 velocity=15; type continuous -> revolute
- joint shoulderPitch_Left: limit (none) -> lower=-3.613 upper=2.042 effort=65 velocity=8; type continuous -> revolute
- joint shoulderPitch_Right: axis 0 -1 0 -> 0 1 0; limit (none) -> lower=-3.613 upper=2.042 effort=65 velocity=8; type continuous -> revolute
- joint shoulderRoll_Left: limit (none) -> lower=-0.628 upper=2.793 effort=65 velocity=8; type continuous -> revolute
- joint shoulderRoll_Right: limit (none) -> lower=-2.793 upper=0.628 effort=65 velocity=8; type continuous -> revolute
- joint shoulderYaw_Left: limit (none) -> lower=-2.583 upper=2.583 effort=65 velocity=8; type continuous -> revolute
- joint shoulderYaw_Right: limit (none) -> lower=-2.583 upper=2.583 effort=65 velocity=8; type continuous -> revolute
- joint waistPitch: axis 0 -1 0 -> 0 1 0; child waistPitch -> waistPitch_link; limit (none) -> lower=-0.663 upper=1.361 effort=110 velocity=8; parent waistRoll -> waistRoll_link; type continuous -> revolute
- joint waistRoll: child waistRoll -> waistRoll_link; limit (none) -> lower=-0.279 upper=0.279 effort=110 velocity=8; type continuous -> revolute
- joint waistYaw: axis 0 0 -1 -> 0 0 1; limit (none) -> lower=-0.829 upper=0.829 effort=110 velocity=8; parent waistPitch -> waistPitch_link; type continuous -> revolute
- joint wristPitch_Left: limit (none) -> lower=-0.96 upper=0.96 effort=6.4 velocity=5; type continuous -> revolute
- joint wristPitch_Right: limit (none) -> lower=-0.96 upper=0.96 effort=6.4 velocity=5; type continuous -> revolute
- joint wristRoll_Left: limit (none) -> lower=-0.96 upper=0.96 effort=6.4 velocity=5; type continuous -> revolute
- joint wristRoll_Right: axis -1 0 0 -> 1 0 0; limit (none) -> lower=-0.96 upper=0.96 effort=6.4 velocity=5; type continuous -> revolute
- joint wristYaw_Left: limit (none) -> lower=-2.67 upper=2.67 effort=6.4 velocity=5; type continuous -> revolute
- joint wristYaw_Right: limit (none) -> lower=-2.67 upper=2.67 effort=6.4 velocity=5; type continuous -> revolute

File: adam_u/adam_u.urdf (robot description, URDF)
Before this commit: robot adam_u, 44 links, 43 joints
Joints:
- joint neckPitch: child neckPitch -> neckPitch_link; parent neckYaw -> neckYaw_link
- joint neckYaw: child neckYaw -> neckYaw_link
- joint waistPitch: child waistPitch -> waistPitch_link; parent waistRoll -> waistRoll_link
- joint waistRoll: child waistRoll -> waistRoll_link
- joint waistYaw: parent waistPitch -> waistPitch_link

Commit message: add imu

File: adam_sp/adam_sp.urdf (robot description, URDF)
Before this commit: robot adam_sp, 54 links, 53 joints
Links:
- added link imu_link, mass 0.001; visual mesh filename=meshes/vn100-0001.dae
Joints:
- added joint imu_joint: type fixed, parent pelvis, child imu_link, origin xyz=0 0 0 rpy=0 0 0

Commit message: add mjcf

File: adam_sp/adam_sp.urdf (robot description, URDF)
Before this commit: robot adam_sp, 55 links, 54 joints
Links:
- link imu_link: geometry 
