Commit message: update models

File: adam_sp/adam_sp.urdf (robot description, URDF)
Before this commit: robot adam_sp, 55 links, 54 joints
Links:
- link L_index_distal: geometry collision mesh filename=meshes_stl_0.25/L_index_distal.STL; visual mesh filename=meshes_stl_0.25/L_index_distal.STL
- link L_index_proximal: geometry collision mesh filename=meshes_stl_0.25/L_index_proximal.STL; visual mesh filename=meshes_stl_0.25/L_index_proximal.STL
- link L_middle_distal: geometry collision mesh filename=meshes_stl_0.25/L_middle_distal.STL; visual mesh filename=meshes_stl_0.25/L_middle_distal.STL
- link L_middle_proximal: geometry collision mesh filename=meshes_stl_0.25/L_middle_proximal.STL; visual mesh filename=meshes_stl_0.25/L_middle_proximal.STL
- link L_pinky_distal: geometry collision mesh filename=meshes_stl_0.25/L_pinky_distal.STL; visual mesh filename=meshes_stl_0.25/L_pinky_distal.STL
- link L_pinky_proximal: geometry collision mesh filename=meshes_stl_0.25/L_pinky_proximal.STL; visual mesh filename=meshes_stl_0.25/L_pinky_proximal.STL
- link L_ring_distal: geometry collision mesh filename=meshes_stl_0.25/L_ring_distal.STL; visual mesh filename=meshes_stl_0.25/L_ring_distal.STL
- link L_ring_proximal: geometry collision mesh filename=meshes_stl_0.25/L_ring_proximal.STL; visual mesh filename=meshes_stl_0.25/L_ring_proximal.STL
- link L_thumb_distal: geometry collision mesh filename=meshes_stl_0.25/L_thumb_distal.STL; visual mesh filename=meshes_stl_0.25/L_thumb_distal.STL
- link L_thumb_intermediate: geometry visual mesh filename=meshes_stl_0.25/L_thumb_intermediate.STL
- link L_thumb_proximal: geometry collision mesh filename=meshes_stl_0.25/L_thumb_proximal.STL; visual mesh filename=meshes_stl_0.25/L_thumb_proximal.STL
- link L_thumb_proximal_base: geometry collision mesh filename=meshes_stl_0.25/L_thumb_proximal_base.STL; visual mesh filename=meshes_stl_0.25/L_thumb_proximal_base.STL
- link R_index_distal: geometry collision mesh filename=meshes_stl_0.25/R_index_distal.STL; visual mesh filename=meshes_stl_0.25/R_index_distal.STL
- link R_index_proximal: geometry collision mesh filename=meshes_stl_0.25/R_index_proximal.STL; visual mesh filename=meshes_stl_0.25/R_index_proximal.STL
- link R_middle_distal: geometry collision mesh filename=meshes_stl_0.25/R_middle_distal.STL; visual mesh filename=meshes_stl_0.25/R_middle_distal.STL
- link R_middle_proximal: geometry collision mesh filename=meshes_stl_0.25/R_middle_proximal.STL; visual mesh filename=meshes_stl_0.25/R_middle_proximal.STL
- link R_pinky_distal: geometry collision mesh filename=meshes_stl_0.25/R_pinky_distal.STL; visual mesh filename=meshes_stl_0.25/R_pinky_distal.STL
- link R_pinky_proximal: geometry collision mesh filename=meshes_stl_0.25/R_pinky_proximal.STL; visual mesh filename=meshes_stl_0.25/R_pinky_proximal.STL
- link R_ring_distal: geometry collision mesh filename=meshes_stl_0.25/R_ring_distal.STL; visual mesh filename=meshes_stl_0.25/R_ring_distal.STL
- link R_ring_proximal: geometry collision mesh filename=meshes_stl_0.25/R_ring_proximal.STL; visual mesh filename=meshes_stl_0.25/R_ring_proximal.STL
- link R_thumb_distal: geometry collision mesh filename=meshes_stl_0.25/R_thumb_distal.STL; visual mesh filename=meshes_stl_0.25/R_thumb_distal.STL
- link R_thumb_intermediate: geometry visual mesh filename=meshes_stl_0.25/R_thumb_intermediate.STL
- link R_thumb_proximal: geometry collision mesh filename=meshes_stl_0.25/R_thumb_proximal.STL; visual mesh filename=meshes_stl_0.25/R_thumb_proximal.STL
- link R_thumb_proximal_base: geometry collision mesh filename=meshes_stl_0.25/R_thumb_proximal_base.STL; visual mesh filename=meshes_stl_0.25/R_thumb_proximal_base.STL
- link anklePitchLeft: geometry collision mesh filename=meshes_stl_0.25/anklePitchLeft.STL; visual mesh filename=meshes_stl_0.25/anklePitchLeft.STL
- link anklePitchRight: geometry collision mesh filename=meshes_stl_0.25/anklePitchRight.STL; visual mesh filename=meshes_stl_0.25/anklePitchRight.STL
- link elbowLeft: geometry collision mesh filename=meshes_stl_0.25/elbowLeft.STL; visual mesh filename=meshes_stl_0.25/elbowLeft.STL
- link elbowRight: geometry collision mesh filename=meshes_stl_0.25/elbowRight.STL; visual mesh filename=meshes_stl_0.25/elbowRight.STL
- link hipPitchLeft: geometry visual mesh filename=meshes_stl_0.25/hipPitchLeft.STL
- link hipPitchRight: geometry visual mesh filename=meshes_stl_0.25/hipPitchRight.STL
- link hipRollLeft: geometry collision mesh filename=meshes_stl_0.25/hipRollLeft.STL; visual mesh filename=meshes_stl_0.25/hipRollLeft.STL
- link hipRollRight: geometry collision mesh filename=meshes_stl_0.25/hipRollRight.STL; visual mesh filename=meshes_stl_0.25/hipRollRight.STL
- link imu_link: mass 0.001 -> None
- link pelvis: geometry collision mesh filename=meshes_stl_0.25/pelvis.STL; visual mesh filename=meshes_stl_0.25/pelvis.STL
- link shinLeft: geometry collision mesh filename=meshes_stl_0.25/shinLeft.STL; visual mesh filename=meshes_stl_0.25/shinLeft.STL
- link shinRight: geometry collision mesh filename=meshes_stl_0.25/shinRight.STL; visual mesh filename=meshes_stl_0.25/shinRight.STL
- link shoulderPitchLeft: geometry collision mesh filename=meshes_stl_0.25/shoulderPitchLeft.STL; visual mesh filename=meshes_stl_0.25/shoulderPitchLeft.STL
- link shoulderPitchRight: geometry collision mesh filename=meshes_stl_0.25/shoulderPitchRight.STL; visual mesh filename=meshes_stl_0.25/shoulderPitchRight.STL
- link shoulderRollLeft: geometry collision mesh filename=meshes_stl_0.25/shoulderRollLeft.STL; visual mesh filename=meshes_stl_0.25/shoulderRollLeft.STL
- link shoulderRollRight: geometry collision mesh filename=meshes_stl_0.25/shoulderRollRight.STL; visual mesh filename=meshes_stl_0.25/shoulderRollRight.STL
- link shoulderYawLeft: geometry collision mesh filename=meshes_stl_0.25/shoulderYawLeft.STL; visual mesh filename=meshes_stl_0.25/shoulderYawLeft.STL
- link shoulderYawRight: geometry collision mesh filename=meshes_stl_0.25/shoulderYawRight.STL; visual mesh filename=meshes_stl_0.25/shoulderYawRight.STL
- link thighLeft: mass 6.43432838 -> 6.43432841; geometry collision mesh filename=meshes_stl_0.25/thighLeft.STL; visual mesh filename=meshes_stl_0.25/thighLeft.STL
- link thighRight: mass 6.43084152 -> 6.43084156; geometry collision mesh filename=meshes_stl_0.25/thighRight.STL; visual mesh filename=meshes_stl_0.25/thighRight.STL
- link toeLeft: geometry collision box size=0.24 0.1 0.02; visual mesh filename=meshes_stl_0.25/toeLeft.STL
- link toeRight: geometry collision box size=0.24 0.1 0.02; visual mesh filename=meshes_stl_0.25/toeRight.STL
- link torso: geometry collision mesh filename=meshes_stl_0.25/torso.STL; visual mesh filename=meshes_stl_0.25/torso.STL
- link waistPitch_link: mass 0.56353776 -> 0.56353777; geometry collision mesh filename=meshes_stl_0.25/waistPitch_link.STL; visual mesh filename=meshes_stl_0.25/waistPitch_link.STL
- link waistRoll_link: geometry visual mesh filename=meshes_stl_0.25/waistRoll_link.STL
- link wristPitchLeft: geometry collision mesh filename=meshes_stl_0.25/wristPitchLeft.STL; visual mesh filename=meshes_stl_0.25/wristPitchLeft.STL
- link wristPitchRight: geometry collision mesh filename=meshes_stl_0.25/wristPitchRight.STL; visual mesh filename=meshes_stl_0.25/wristPitchRight.STL
- link wristRollLeft: geometry visual mesh filename=meshes_stl_0.25/wristRollLeft.STL
- link wristRollRight: geometry visual mesh filename=meshes_stl_0.25/wristRollRight.STL
- link wristYawLeft: geometry collision mesh filename=meshes_stl_0.25/wristYawLeft.STL; visual mesh filename=meshes_stl_0.25/wristYawLeft.STL
- link wristYawRight: geometry collision mesh filename=meshes_stl_0.25/wristYawRight.STL; visual mesh filename=meshes_stl_0.25/wristYawRight.STL

File: adam_sp_pro/adam_sp_pro.urdf (robot description, URDF)
Before this commit: robot adam_sp_pro, 56 links, 55 joints
Links:
- added link imu_link
- link L_thumb_intermediate: geometry visual mesh filename=meshes_stl_0.25/L_thumb_intermediate.STL
- link R_thumb_intermediate: geometry visual mesh filename=meshes_stl_0.25/R_thumb_intermediate.STL
- link hipPitchLeft: geometry visual mesh filename=meshes_stl_0.25/hipPitchLeft.STL
- link hipPitchRight: geometry visual mesh filename=meshes_stl_0.25/hipPitchRight.STL
- link toeLeft: geometry collision box size=0.24 0.1 0.02; visual mesh filename=meshes_stl_0.25/toeLeft.STL
- link toeRight: geometry collision box size=0.24 0.1 0.02; visual mesh filename=meshes_stl_0.25/toeRight.STL
- link wristRollLeft: geometry visual mesh filename=meshes_stl_0.25/wristRollLeft.STL
- link wristRollRight: geometry visual mesh filename=meshes_stl_0.25/wristRollRight.STL
Joints:
- added joint imu_joint: type fixed, parent pelvis, child imu_link, origin xyz=0 0 0 rpy=0 0 0

File: adam_u/adam_u.urdf (robot description, URDF)
Before this commit: robot adam_u, 44 links, 43 joints
Links:
- link L_thumb_intermediate: geometry visual mesh filename=meshes_dae/L_thumb_intermediate.dae
- link R_thumb_intermediate: geometry visual mesh filename=meshes_dae/R_thumb_intermediate.dae
- link elbowLeft: mass 0.87761532 -> 0.91770702
- link elbowRight: mass 0.87761532 -> 0.91770702
- link neckPitch_link: mass 0.99740875 -> 0.95620414; geometry collision mesh filename=meshes_stl_0.25/neckPitch_link.STL; visual mesh filename=meshes_dae/neckPitch.dae
- link neckYaw_link: mass 0.41242410 -> 0.39916798; geometry collision mesh filename=meshes_stl_0.25/neckYaw_link.STL; visual mesh filename=meshes_dae/neckYaw.dae
- link shoulderPitchLeft: mass 0.21653557 -> 0.21614811
- link shoulderPitchRight: mass 0.21653557 -> 0.21648747
- link shoulderRollLeft: mass 0.74622709 -> 1.07881773
- link shoulderRollRight: mass 0.74506856 -> 1.08875448
- link shoulderYawLeft: mass 0.76573936 -> 0.90142027
- link shoulderYawRight: mass 0.76530592 -> 0.90139273
- link torso: mass 12.22987423 -> 12.73336771
- link waistPitch_link: mass 0.56353776 -> 0.56353777; geometry collision mesh filename=meshes_stl_0.25/waistPitch_link.STL; visual mesh filename=meshes_dae/waistPitch.dae
- link waistRoll_link: geometry collision mesh filename=meshes_stl_0.25/waistRoll_link.STL; visual mesh filename=meshes_dae/waistRoll.dae
- link wristRollLeft: geometry visual mesh filename=meshes_dae/wristRollLeft.dae
- link wristRollRight: geometry visual mesh filename=meshes_dae/wristRollRight.dae
Joints:
- joint L_index_DIP_joint: origin xyz=0 -0.0011127 -0.031981 rpy=0 0 0 -> xyz=0 -0.00111268989731944 -0.0319806491677784 rpy=0 0 0
- joint L_index_MCP_joint: origin xyz=0.026942 0.0095 -0.11498 rpy=0 -0.05236 0 -> xyz=0.0269420472022218 0.00950000000154763 -0.114975331627829 rpy=0 -0.0523598774782631 0
- joint L_middle_DIP_joint: origin xyz=0 -0.0029374 -0.031865 rpy=0 0 0 -> xyz=0 -0.00293735370583337 -0.0318649015879072 rpy=0 0 0
- joint L_middle_MCP_joint: origin xyz=0.008 0.0145 -0.128 rpy=0 0 0 -> xyz=0.00799999998838565 0.0144999999999475 -0.128000000000728 rpy=0 0 0
- joint L_pinky_DIP_joint: origin xyz=0 -0.0011127 -0.031981 rpy=0 0 0 -> xyz=0 -0.00111268989776986 -0.0319806491677628 rpy=0 0 0
- joint L_pinky_MCP_joint: origin xyz=-0.030194 0.0045 -0.11287 rpy=0 0.12217 0 -> xyz=-0.0301936481908677 0.00449999999694281 -0.11286583072711 rpy=0 0.12217304772112 0
- joint L_ring_DIP_joint: origin xyz=0 -0.0011127 -0.031981 rpy=0 0 0 -> xyz=0 -0.00111268989759014 -0.0319806491677691 rpy=0 0 0
- joint L_ring_MCP_joint: origin xyz=-0.010942 0.0095 -0.11998 rpy=0 0.05236 0 -> xyz=-0.0109420472229284 0.00949999999845705 -0.119975331624717 rpy=0 0.052359877641387 0
- joint L_thumb_DIP_joint: origin xyz=0.016468 0 -0.015461 rpy=0 0 0 -> xyz=0.0164679343341741 0 -0.0154614727230483 rpy=0 0 0
- joint L_thumb_MCP_joint1: origin xyz=0.0245 -0.01 -0.047 rpy=0 0 0 -> xyz=0.0244999999969742 -0.0099999999982788 -0.0470000000019433 rpy=0 0 0
- joint L_thumb_MCP_joint2: origin xyz=0.011954 -0.0010497 0 rpy=0 0 -0.087585 -> xyz=0.011954002456522 -0.00104967865057148 0 rpy=0 0 -0.0875851578962738
- joint L_thumb_PIP_joint: origin xyz=0.044289 0 -0.037663 rpy=0 0 0 -> xyz=0.0442885641132063 0 -0.0376632856876562 rpy=0 0 0
- joint R_index_DIP_joint: origin xyz=0 0.0011127 -0.031981 rpy=0 0 0 -> xyz=0 0.00111268989722751 -0.0319806491677816 rpy=0 0 0
- joint R_index_MCP_joint: origin xyz=0.026942 -0.0095 -0.11498 rpy=0 -0.05236 0 -> xyz=0.0269420472120735 -0.00950000000009146 -0.114975331625641 rpy=0 -0.0523598775568891 0
- joint R_middle_DIP_joint: origin xyz=0 0.0029374 -0.031865 rpy=0 0 0 -> xyz=0 0.00293735370559906 -0.0318649015879289 rpy=0 0 0
- joint R_middle_MCP_joint: origin xyz=0.008 -0.0145 -0.128 rpy=0 0 0 -> xyz=0.00799999999968861 -0.0145000000002054 -0.127999999999992 rpy=0 0 0
- joint R_pinky_DIP_joint: origin xyz=0 0.0011127 -0.031981 rpy=0 0 0 -> xyz=0 0.00111268989720342 -0.0319806491677825 rpy=0 0 0
- joint R_pinky_MCP_joint: origin xyz=-0.030194 -0.0045 -0.11287 rpy=0 0.12217 0 -> xyz=-0.0301936481816091 -0.00450000000035261 -0.112865830729451 rpy=0 0.122173047642494 0
- joint R_ring_DIP_joint: origin xyz=0 0.0011127 -0.031981 rpy=0 0 0 -> xyz=0 0.00111268989721214 -0.0319806491677822 rpy=0 0 0
- joint R_ring_MCP_joint: origin xyz=-0.010942 -0.0095 -0.11998 rpy=0 0.05236 0 -> xyz=-0.0109420472126836 -0.00950000000027432 -0.119975331625507 rpy=0 0.0523598775627611 0
- joint R_thumb_DIP_joint: origin xyz=0.016468 0 -0.015461 rpy=0 0 0 -> xyz=0.0164679343353944 0 -0.0154614727217485 rpy=0 0 0
- joint R_thumb_MCP_joint1: origin xyz=0.0245 0.01 -0.047 rpy=0 0 0 -> xyz=0.0244999999998152 0.0100000000000263 -0.0470000000000906 rpy=0 0 0
- joint R_thumb_MCP_joint2: origin xyz=0.011954 0.0010497 0 rpy=0 0 0.087585 -> xyz=0.0119540024564323 0.00104967865159283 0 rpy=0 0 0.0875851579817108
- joint R_thumb_PIP_joint: origin xyz=0.044289 0 -0.037663 rpy=0 0 0 -> xyz=0.044288564116179 0 -0.0376632856841606 rpy=0 0 0
- joint elbow_Left: origin xyz=0 -0.0285 -0.20415 rpy=0 0 0 -> xyz=0 -0.0285000000009982 -0.182950000001738 rpy=0 0 0
- joint elbow_Right: origin xyz=0 0.0285 -0.20415 rpy=0 0 0 -> xyz=0 0.0284999999998828 -0.182950000001922 rpy=0 0 0
- joint neckPitch: origin xyz=0.0316 0.02 0.14595 rpy=0 0 0 -> xyz=0.0316000000000086 0.0199499999999967 0.145949999999989 rpy=0 0 0
- joint neckYaw: origin xyz=-0.013 0 0.29855 rpy=0 0 0 -> xyz=-0.0130000000000059 0 0.298550000000013 rpy=0 0 0
- joint shoulderPitch_Left: origin xyz=0 0.16049 0.25755 rpy=0.34907 0 0 -> xyz=0 0.165093970689425 0.259229560594865 rpy=0.349065850393456 0 0
- joint shoulderPitch_Right: origin xyz=0 -0.16049 0.25755 rpy=-0.34907 0 0 -> xyz=0 -0.165093970689321 0.259229560595242 rpy=-0.349065850398898 0 0
- joint shoulderRoll_Left: origin xyz=0.0335 0.0435 0 rpy=-0.34907 0 0 -> xyz=0.036199999996826 0.0434999999975074 0 rpy=-0.349065850393456 0 0
- joint shoulderRoll_Right: origin xyz=0.0335 -0.0435 0 rpy=0.34907 0 0 -> xyz=0.036199999639011 -0.0435000000171988 0 rpy=0.349065850398898 0 0
- joint shoulderYaw_Left: origin xyz=-0.0335 0.034 -0.0585 rpy=0 0 0 -> xyz=-0.0361999999622004 0.0340000000110588 -0.0796999999903454 rpy=0 0 0
- joint shoulderYaw_Right: origin xyz=-0.0335 -0.034 -0.0585 rpy=0 0 0 -> xyz=-0.0361999996389017 -0.0339999999996759 -0.0797000000498751 rpy=0 0 0
- joint waistYaw: origin xyz=0 0.0005 0.053 rpy=0 0 0 -> xyz=0 0.000500000000007081 0.05299999999999 rpy=0 0 0
- joint wristPitch_Left: origin xyz=0 0 -0.2017 rpy=0 0 0 -> xyz=0 0 -0.201699999999994 rpy=0 0 0
- joint wristPitch_Right: origin xyz=0 0 -0.2017 rpy=0 0 0 -> xyz=0 0 -0.201699999999861 rpy=0 0 0
- joint wristYaw_Left: origin xyz=-0.025 0.0285 -0.0729 rpy=0 0 0 -> xyz=-0.0250000000083053 0.028499999997574 -0.0728999999980683 rpy=0 0 0
- joint wristYaw_Right: origin xyz=-0.025 -0.0285 -0.0729 rpy=0 0 0 -> xyz=-0.0249999999999065 -0.0285000000002922 -0.0728999999999894 rpy=0 0 0
