Commit message: update adam_u urdf

File: adam_u/adam_u.urdf (robot description, URDF)
Before this commit: robot adam_u, 44 links, 43 joints
Links:
- link L_index_distal: geometry collision mesh filename=meshes_stl_0.25/L_index_distal.STL; visual mesh filename=meshes_dae/L_index_distal.dae
- link L_index_proximal: geometry collision mesh filename=meshes_stl_0.25/L_index_proximal.STL; visual mesh filename=meshes_dae/L_index_proximal.dae
- link L_middle_distal: geometry collision mesh filename=meshes_stl_0.25/L_middle_distal.STL; visual mesh filename=meshes_dae/L_middle_distal.dae
- link L_middle_proximal: geometry collision mesh filename=meshes_stl_0.25/L_middle_proximal.STL; visual mesh filename=meshes_dae/L_middle_proximal.dae
- link L_pinky_distal: geometry collision mesh filename=meshes_stl_0.25/L_pinky_distal.STL; visual mesh filename=meshes_dae/L_pinky_distal.dae
- link L_pinky_proximal: geometry collision mesh filename=meshes_stl_0.25/L_pinky_proximal.STL; visual mesh filename=meshes_dae/L_pinky_proximal.dae
- link L_ring_distal: geometry collision mesh filename=meshes_stl_0.25/L_ring_distal.STL; visual mesh filename=meshes_dae/L_ring_distal.dae
- link L_ring_proximal: geometry collision mesh filename=meshes_stl_0.25/L_ring_proximal.STL; visual mesh filename=meshes_dae/L_ring_proximal.dae
- link L_thumb_distal: geometry collision mesh filename=meshes_stl_0.25/L_thumb_distal.STL; visual mesh filename=meshes_dae/L_thumb_distal.dae
- link L_thumb_intermediate: geometry collision mesh filename=meshes_stl_0.25/L_thumb_intermediate.STL; visual mesh filename=meshes_dae/L_thumb_intermediate.dae
- link L_thumb_proximal: geometry collision mesh filename=meshes_stl_0.25/L_thumb_proximal.STL; visual mesh filename=meshes_dae/L_thumb_proximal.dae
- link L_thumb_proximal_base: geometry collision mesh filename=meshes_stl_0.25/L_thumb_proximal_base.STL; visual mesh filename=meshes_dae/L_thumb_proximal_base.dae
- link R_index_distal: geometry collision mesh filename=meshes_stl_0.25/R_index_distal.STL; visual mesh filename=meshes_dae/R_index_distal.dae
- link R_index_proximal: geometry collision mesh filename=meshes_stl_0.25/R_index_proximal.STL; visual mesh filename=meshes_dae/R_index_proximal.dae
- link R_middle_distal: geometry collision mesh filename=meshes_stl_0.25/R_middle_distal.STL; visual mesh filename=meshes_dae/R_middle_distal.dae
- link R_middle_proximal: geometry collision mesh filename=meshes_stl_0.25/R_middle_proximal.STL; visual mesh filename=meshes_dae/R_middle_proximal.dae
- link R_pinky_distal: geometry collision mesh filename=meshes_stl_0.25/R_pinky_distal.STL; visual mesh filename=meshes_dae/R_pinky_distal.dae
- link R_pinky_proximal: geometry collision mesh filename=meshes_stl_0.25/R_pinky_proximal.STL; visual mesh filename=meshes_dae/R_pinky_proximal.dae
- link R_ring_distal: geometry collision mesh filename=meshes_stl_0.25/R_ring_distal.STL; visual mesh filename=meshes_dae/R_ring_distal.dae
- link R_ring_proximal: geometry collision mesh filename=meshes_stl_0.25/R_ring_proximal.STL; visual mesh filename=meshes_dae/R_ring_proximal.dae
- link R_thumb_distal: geometry collision mesh filename=meshes_stl_0.25/R_thumb_distal.STL; visual mesh filename=meshes_dae/R_thumb_distal.dae
- link R_thumb_intermediate: geometry collision mesh filename=meshes_stl_0.25/R_thumb_intermediate.STL; visual mesh filename=meshes_dae/R_thumb_intermediate.dae
- link R_thumb_proximal: geometry collision mesh filename=meshes_stl_0.25/R_thumb_proximal.STL; visual mesh filename=meshes_dae/R_thumb_proximal.dae
- link R_thumb_proximal_base: geometry collision mesh filename=meshes_stl_0.25/R_thumb_proximal_base.STL; visual mesh filename=meshes_dae/R_thumb_proximal_base.dae
- link elbowLeft: geometry collision mesh filename=meshes_stl_0.25/elbowLeft.STL; visual mesh filename=meshes_dae/elbowLeft.dae
- link elbowRight: geometry collision mesh filename=meshes_stl_0.25/elbowRight.STL; visual mesh filename=meshes_dae/elbowRight.dae
- link lifting_Columns: geometry collision mesh filename=meshes_stl_0.25/lifting_Columns.STL; visual mesh filename=meshes_dae/lifting_Columns.dae
- link neckPitch: geometry collision mesh filename=meshes_stl_0.25/neckPitch.STL; visual mesh filename=meshes_dae/neckPitch.dae
- link neckYaw: geometry collision mesh filename=meshes_stl_0.25/neckYaw.STL; visual mesh filename=meshes_dae/neckYaw.dae
- link shoulderPitchLeft: geometry collision mesh filename=meshes_stl_0.25/shoulderPitchLeft.STL; visual mesh filename=meshes_dae/shoulderPitchLeft.dae
- link shoulderPitchRight: geometry collision mesh filename=meshes_stl_0.25/shoulderPitchRight.STL; visual mesh filename=meshes_dae/shoulderPitchRight.dae
- link shoulderRollLeft: geometry collision mesh filename=meshes_stl_0.25/shoulderRollLeft.STL; visual mesh filename=meshes_dae/shoulderRollLeft.dae
- link shoulderRollRight: geometry collision mesh filename=meshes_stl_0.25/shoulderRollRight.STL; visual mesh filename=meshes_dae/shoulderRollRight.dae
- link shoulderYawLeft: geometry collision mesh filename=meshes_stl_0.25/shoulderYawLeft.STL; visual mesh filename=meshes_dae/shoulderYawLeft.dae
- link shoulderYawRight: geometry collision mesh filename=meshes_stl_0.25/shoulderYawRight.STL; visual mesh filename=meshes_dae/shoulderYawRight.dae
- link torso: geometry collision mesh filename=meshes_stl_0.25/torso.STL; visual mesh filename=meshes_dae/torso.dae
- link waistPitch: geometry collision mesh filename=meshes_stl_0.25/waistPitch.STL; visual mesh filename=meshes_dae/waistPitch.dae
- link waistRoll: geometry collision mesh filename=meshes_stl_0.25/waistRoll.STL; visual mesh filename=meshes_dae/waistRoll.dae
- link wristPitchLeft: geometry collision mesh filename=meshes_stl_0.25/wristPitchLeft.STL; visual mesh filename=meshes_dae/wristPitchLeft.dae
- link wristPitchRight: geometry collision mesh filename=meshes_stl_0.25/wristPitchRight.STL; visual mesh filename=meshes_dae/wristPitchRight.dae
- link wristRollLeft: geometry collision mesh filename=meshes_stl_0.25/wristRollLeft.STL; visual mesh filename=meshes_dae/wristRollLeft.dae
- link wristRollRight: geometry collision mesh filename=meshes_stl_0.25/wristRollRight.STL; visual mesh filename=meshes_dae/wristRollRight.dae
- link wristYawLeft: geometry collision mesh filename=meshes_stl_0.25/wristYawLeft.STL; visual mesh filename=meshes_dae/wristYawLeft.dae
- link wristYawRight: geometry collision mesh filename=meshes_stl_0.25/wristYawRight.STL; visual mesh filename=meshes_dae/wristYawRight.dae

Commit message: fix inertia

File: adam_u/adam_u.urdf (robot description, URDF)
Before this commit: robot adam_u, 44 links, 43 joints
Links:
- link L_index_distal: geometry collision mesh filename=meshes_stl_0.25/L_index_distal.STL; visual mesh filename=meshes_stl_0.25/L_index_distal.STL
- link L_index_proximal: geometry collision mesh filename=meshes_stl_0.25/L_index_proximal.STL; visual mesh filename=meshes_stl_0.25/L_index_proximal.STL
- link L_middle_distal: geometry collision mesh filename=meshes_stl_0.25/L_middle_distal.STL; visual mesh filename=meshes_stl_0.25/L_middle_distal.STL
- link L_middle_proximal: geometry collision mesh filename=meshes_stl_0.25/L_middle_proximal.STL; visual mesh filename=meshes_stl_0.25/L_middle_proximal.STL
- link L_pinky_distal: geometry collision mesh filename=meshes_stl_0.25/L_pinky_distal.STL; visual mesh filename=meshes_stl_0.25/L_pinky_distal.STL
- link L_pinky_proximal: geometry collision mesh filename=meshes_stl_0.25/L_pinky_proximal.STL; visual mesh filename=meshes_stl_0.25/L_pinky_proximal.STL
- link L_ring_distal: geometry collision mesh filename=meshes_stl_0.25/L_ring_distal.STL; visual mesh filename=meshes_stl_0.25/L_ring_distal.STL
- link L_ring_proximal: geometry collision mesh filename=meshes_stl_0.25/L_ring_proximal.STL; visual mesh filename=meshes_stl_0.25/L_ring_proximal.STL
- link L_thumb_distal: geometry collision mesh filename=meshes_stl_0.25/L_thumb_distal.STL; visual mesh filename=meshes_stl_0.25/L_thumb_distal.STL
- link L_thumb_intermediate: geometry visual mesh filename=meshes_stl_0.25/L_thumb_intermediate.STL
- link L_thumb_proximal: geometry collision mesh filename=meshes_stl_0.25/L_thumb_proximal.STL; visual mesh filename=meshes_stl_0.25/L_thumb_proximal.STL
- link L_thumb_proximal_base: geometry collision mesh filename=meshes_stl_0.25/L_thumb_proximal_base.STL; visual mesh filename=meshes_stl_0.25/L_thumb_proximal_base.STL
- link R_index_distal: geometry collision mesh filename=meshes_stl_0.25/R_index_distal.STL; visual mesh filename=meshes_stl_0.25/R_index_distal.STL
- link R_index_proximal: geometry collision mesh filename=meshes_stl_0.25/R_index_proximal.STL; visual mesh filename=meshes_stl_0.25/R_index_proximal.STL
- link R_middle_distal: geometry collision mesh filename=meshes_stl_0.25/R_middle_distal.STL; visual mesh filename=meshes_stl_0.25/R_middle_distal.STL
- link R_middle_proximal: geometry collision mesh filename=meshes_stl_0.25/R_middle_proximal.STL; visual mesh filename=meshes_stl_0.25/R_middle_proximal.STL
- link R_pinky_distal: geometry collision mesh filename=meshes_stl_0.25/R_pinky_distal.STL; visual mesh filename=meshes_stl_0.25/R_pinky_distal.STL
- link R_pinky_proximal: geometry collision mesh filename=meshes_stl_0.25/R_pinky_proximal.STL; visual mesh filename=meshes_stl_0.25/R_pinky_proximal.STL
- link R_ring_distal: geometry collision mesh filename=meshes_stl_0.25/R_ring_distal.STL; visual mesh filename=meshes_stl_0.25/R_ring_distal.STL
- link R_ring_proximal: geometry collision mesh filename=meshes_stl_0.25/R_ring_proximal.STL; visual mesh filename=meshes_stl_0.25/R_ring_proximal.STL
- link R_thumb_distal: geometry collision mesh filename=meshes_stl_0.25/R_thumb_distal.STL; visual mesh filename=meshes_stl_0.25/R_thumb_distal.STL
- link R_thumb_intermediate: geometry visual mesh filename=meshes_stl_0.25/R_thumb_intermediate.STL
- link R_thumb_proximal: geometry collision mesh filename=meshes_stl_0.25/R_thumb_proximal.STL; visual mesh filename=meshes_stl_0.25/R_thumb_proximal.STL
- link R_thumb_proximal_base: geometry collision mesh filename=meshes_stl_0.25/R_thumb_proximal_base.STL; visual mesh filename=meshes_stl_0.25/R_thumb_proximal_base.STL
- link elbowLeft: geometry collision mesh filename=meshes_stl_0.25/elbowLeft.STL; visual mesh filename=meshes_stl_0.25/elbowLeft.STL
- link elbowRight: geometry collision mesh filename=meshes_stl_0.25/elbowRight.STL; visual mesh filename=meshes_stl_0.25/elbowRight.STL
- link lifting_Columns: geometry collision mesh filename=meshes_stl_0.25/lifting_Columns.STL; visual mesh filename=meshes_stl_0.25/lifting_Columns.STL
- link neckPitch_link: geometry collision mesh filename=meshes_stl_0.25/neckPitch_link.STL; visual mesh filename=meshes_stl_0.25/neckPitch_link.STL
- link neckYaw_link: geometry collision mesh filename=meshes_stl_0.25/neckYaw_link.STL; visual mesh filename=meshes_stl_0.25/neckYaw_link.STL
- link shoulderPitchLeft: geometry collision mesh filename=meshes_stl_0.25/shoulderPitchLeft.STL; visual mesh filename=meshes_stl_0.25/shoulderPitchLeft.STL
- link shoulderPitchRight: geometry collision mesh filename=meshes_stl_0.25/shoulderPitchRight.STL; visual mesh filename=meshes_stl_0.25/shoulderPitchRight.STL
- link shoulderRollLeft: geometry collision mesh filename=meshes_stl_0.25/shoulderRollLeft.STL; visual mesh filename=meshes_stl_0.25/shoulderRollLeft.STL
- link shoulderRollRight: geometry collision mesh filename=meshes_stl_0.25/shoulderRollRight.STL; visual mesh filename=meshes_stl_0.25/shoulderRollRight.STL
- link shoulderYawLeft: geometry collision mesh filename=meshes_stl_0.25/shoulderYawLeft.STL; visual mesh filename=meshes_stl_0.25/shoulderYawLeft.STL
- link shoulderYawRight: geometry collision mesh filename=meshes_stl_0.25/shoulderYawRight.STL; visual mesh filename=meshes_stl_0.25/shoulderYawRight.STL
- link torso: geometry collision mesh filename=meshes_stl_0.25/torso.STL; visual mesh filename=meshes_stl_0.25/torso.STL
- link waistPitch_link: geometry collision mesh filename=meshes_stl_0.25/waistPitch_link.STL; visual mesh filename=meshes_stl_0.25/waistPitch_link.STL
- link waistRoll_link: geometry collision mesh filename=meshes_stl_0.25/waistRoll_link.STL; visual mesh filename=meshes_stl_0.25/waistRoll_link.STL
- link wristPitchLeft: geometry collision mesh filename=meshes_stl_0.25/wristPitchLeft.STL; visual mesh filename=meshes_stl_0.25/wristPitchLeft.STL
- link wristPitchRight: geometry collision mesh filename=meshes_stl_0.25/wristPitchRight.STL; visual mesh filename=meshes_stl_0.25/wristPitchRight.STL
- link wristRollLeft: geometry visual mesh filename=meshes_stl_0.25/wristRollLeft.STL
- link wristRollRight: geometry visual mesh filename=meshes_stl_0.25/wristRollRight.STL
- link wristYawLeft: geometry collision mesh filename=meshes_stl_0.25/wristYawLeft.STL; visual mesh filename=meshes_stl_0.25/wristYawLeft.STL
- link wristYawRight: geometry collision mesh filename=meshes_stl_0.25/wristYawRight.STL; visual mesh filename=meshes_stl_0.25/wristYawRight.STL
