Commit message: Add adam_u_pro_max

File: adam_sp_pro/adam_sp_pro.urdf (robot description, URDF)
Before this commit: robot adam_sp_pro, 57 links, 56 joints
Links:
- link waistRoll_link: geometry visual mesh filename=meshes_stl_0.25/waistRoll_link.STL

Commit message: add adam_sp_pro dae

File: adam_sp_pro/adam_sp_pro.urdf (robot description, URDF)
Before this commit: robot adam_sp_pro, 57 links, 56 joints
Links:
- link L_index_distal: geometry collision mesh filename=meshes_stl_0.25/L_index_distal.STL; visual mesh filename=meshes_dae/L_index_distal.dae
- link L_index_proximal: geometry collision mesh filename=meshes_stl_0.25/L_index_proximal.STL; visual mesh filename=meshes_dae/L_index_proximal.dae
- link L_middle_distal: geometry collision mesh filename=meshes_stl_0.25/L_middle_distal.STL; visual mesh filename=meshes_dae/L_middle_distal.dae
- link L_middle_proximal: geometry collision mesh filename=meshes_stl_0.25/L_middle_proximal.STL; visual mesh filename=meshes_dae/L_middle_proximal.dae
- link L_pinky_distal: geometry collision mesh filename=meshes_stl_0.25/L_pinky_distal.STL; visual mesh filename=meshes_dae/L_pinky_distal.dae
- link L_pinky_proximal: geometry collision mesh filename=meshes_stl_0.25/L_pinky_proximal.STL; visual mesh filename=meshes_dae/L_pinky_proximal.dae
- link L_ring_distal: geometry collision mesh filename=meshes_stl_0.25/L_ring_distal.STL; visual mesh filename=meshes_dae/L_ring_distal.dae
- link L_ring_proximal: geometry collision mesh filename=meshes_stl_0.25/L_ring_proximal.STL; visual mesh filename=meshes_dae/L_ring_proximal.dae
- link L_thumb_distal: geometry collision mesh filename=meshes_stl_0.25/L_thumb_distal.STL; visual mesh filename=meshes_dae/L_thumb_distal.dae
- link L_thumb_intermediate: geometry visual mesh filename=meshes_dae/L_thumb_intermediate.dae
- link L_thumb_proximal: geometry collision mesh filename=meshes_stl_0.25/L_thumb_proximal.STL; visual mesh filename=meshes_dae/L_thumb_proximal.dae
- link L_thumb_proximal_base: geometry collision mesh filename=meshes_stl_0.25/L_thumb_proximal_base.STL; visual mesh filename=meshes_dae/L_thumb_proximal_base.dae
- link R_index_distal: geometry collision mesh filename=meshes_stl_0.25/R_index_distal.STL; visual mesh filename=meshes_dae/R_index_distal.dae
- link R_index_proximal: geometry collision mesh filename=meshes_stl_0.25/R_index_proximal.STL; visual mesh filename=meshes_dae/R_index_proximal.dae
- link R_middle_distal: geometry collision mesh filename=meshes_stl_0.25/R_middle_distal.STL; visual mesh filename=meshes_dae/R_middle_distal.dae
- link R_middle_proximal: geometry collision mesh filename=meshes_stl_0.25/R_middle_proximal.STL; visual mesh filename=meshes_dae/R_middle_proximal.dae
- link R_pinky_distal: geometry collision mesh filename=meshes_stl_0.25/R_pinky_distal.STL; visual mesh filename=meshes_dae/R_pinky_distal.dae
- link R_pinky_proximal: geometry collision mesh filename=meshes_stl_0.25/R_pinky_proximal.STL; visual mesh filename=meshes_dae/R_pinky_proximal.dae
- link R_ring_distal: geometry collision mesh filename=meshes_stl_0.25/R_ring_distal.STL; visual mesh filename=meshes_dae/R_ring_distal.dae
- link R_ring_proximal: geometry collision mesh filename=meshes_stl_0.25/R_ring_proximal.STL; visual mesh filename=meshes_dae/R_ring_proximal.dae
- link R_thumb_distal: geometry collision mesh filename=meshes_stl_0.25/R_thumb_distal.STL; visual mesh filename=meshes_dae/R_thumb_distal.dae
- link R_thumb_intermediate: geometry visual mesh filename=meshes_dae/R_thumb_intermediate.dae
- link R_thumb_proximal: geometry collision mesh filename=meshes_stl_0.25/R_thumb_proximal.STL; visual mesh filename=meshes_dae/R_thumb_proximal.dae
- link R_thumb_proximal_base: geometry collision mesh filename=meshes_stl_0.25/R_thumb_proximal_base.STL; visual mesh filename=meshes_dae/R_thumb_proximal_base.dae
- link anklePitchLeft: geometry collision mesh filename=meshes_stl_0.25/anklePitchLeft.STL; visual mesh filename=meshes_dae/anklePitchLeft.dae
- link anklePitchRight: geometry collision mesh filename=meshes_stl_0.25/anklePitchRight.STL; visual mesh filename=meshes_dae/anklePitchRight.dae
- link elbowLeft: geometry collision mesh filename=meshes_stl_0.25/elbowLeft.STL; visual mesh filename=meshes_dae/elbowLeft.dae
- link elbowRight: geometry collision mesh filename=meshes_stl_0.25/elbowRight.STL; visual mesh filename=meshes_dae/elbowRight.dae
- link hipPitchLeft: geometry visual mesh filename=meshes_dae/hipPitchLeft.dae
- link hipPitchRight: geometry visual mesh filename=meshes_dae/hipPitchRight.dae
- link hipRollLeft: geometry collision mesh filename=meshes_stl_0.25/hipRollLeft.STL; visual mesh filename=meshes_dae/hipRollLeft.dae
- link hipRollRight: geometry collision mesh filename=meshes_stl_0.25/hipRollRight.STL; visual mesh filename=meshes_dae/hipRollRight.dae
- link neckPitch_link: geometry collision mesh filename=meshes_stl_0.25/neckPitch_link.STL; visual mesh filename=meshes_dae/neckPitch_link.dae
- link neckYaw_link: geometry collision mesh filename=meshes_stl_0.25/neckYaw_link.STL; visual mesh filename=meshes_dae/neckYaw_link.dae
- link pelvis: geometry collision mesh filename=meshes_stl_0.25/pelvis.STL; visual mesh filename=meshes_dae/pelvis.dae
- link shinLeft: geometry collision mesh filename=meshes_stl_0.25/shinLeft.STL; visual mesh filename=meshes_dae/shinLeft.dae
- link shinRight: geometry collision mesh filename=meshes_stl_0.25/shinRight.STL; visual mesh filename=meshes_dae/shinRight.dae
- link shoulderPitchLeft: geometry collision mesh filename=meshes_stl_0.25/shoulderPitchLeft.STL; visual mesh filename=meshes_dae/shoulderPitchLeft.dae
- link shoulderPitchRight: geometry collision mesh filename=meshes_stl_0.25/shoulderPitchRight.STL; visual mesh filename=meshes_dae/shoulderPitchRight.dae
- link shoulderRollLeft: geometry collision mesh filename=meshes_stl_0.25/shoulderRollLeft.STL; visual mesh filename=meshes_dae/shoulderRollLeft.dae
- link shoulderRollRight: geometry collision mesh filename=meshes_stl_0.25/shoulderRollRight.STL; visual mesh filename=meshes_dae/shoulderRollRight.dae
- link shoulderYawLeft: geometry collision mesh filename=meshes_stl_0.25/shoulderYawLeft.STL; visual mesh filename=meshes_dae/shoulderYawLeft.dae
- link shoulderYawRight: geometry collision mesh filename=meshes_stl_0.25/shoulderYawRight.STL; visual mesh filename=meshes_dae/shoulderYawRight.dae
- link thighLeft: geometry collision mesh filename=meshes_stl_0.25/thighLeft.STL; visual mesh filename=meshes_dae/thighLeft.dae
- link thighRight: geometry collision mesh filename=meshes_stl_0.25/thighRight.STL; visual mesh filename=meshes_dae/thighRight.dae
- link toeLeft: geometry collision box size=0.24 0.1 0.02; visual mesh filename=meshes_dae/toeLeft.dae
- link toeRight: geometry collision box size=0.24 0.1 0.02; visual mesh filename=meshes_dae/toeRight.dae
- link torso: geometry collision mesh filename=meshes_stl_0.25/torso.STL; visual mesh filename=meshes_dae/torso.dae
- link waistPitch_link: geometry collision mesh filename=meshes_stl_0.25/waistPitch_link.STL; visual mesh filename=meshes_dae/waistPitch_link.dae
- link waistRoll_link: geometry visual mesh filename=meshes_dae/waistRoll_link.dae
- link wristPitchLeft: geometry collision mesh filename=meshes_stl_0.25/wristPitchLeft.STL; visual mesh filename=meshes_dae/wristPitchLeft.dae
- link wristPitchRight: geometry collision mesh filename=meshes_stl_0.25/wristPitchRight.STL; visual mesh filename=meshes_dae/wristPitchRight.dae
- link wristRollLeft: geometry visual mesh filename=meshes_dae/wristRollLeft.dae
- link wristRollRight: geometry visual mesh filename=meshes_dae/wristRollRight.dae
- link wristYawLeft: geometry collision mesh filename=meshes_stl_0.25/wristYawLeft.STL; visual mesh filename=meshes_dae/wristYawLeft.dae
- link wristYawRight: geometry collision mesh filename=meshes_stl_0.25/wristYawRight.STL; visual mesh filename=meshes_dae/wristYawRight.dae
