Commit message: add camera

File: adam_pro/adam_pro.urdf (robot description, URDF)
Before this commit: robot adam_pro, 57 links, 56 joints
Links:
- added link left_zed_link
- added link right_zed_link
Joints:
- added joint left_zed_joint: type fixed, parent neckPitch_link, child left_zed_link, origin xyz=0.096 0.0118 0.0407 rpy=0 0 0
- added joint right_zed_joint: type fixed, parent neckPitch_link, child right_zed_link, origin xyz=0.096 -0.0517 0.0407 rpy=0 0 0

File: adam_u/adam_u.urdf (robot description, URDF)
Before this commit: robot adam_u, 44 links, 43 joints
Links:
- added link left_zed_link
- added link right_zed_link
Joints:
- added joint left_zed_joint: type fixed, parent neckPitch_link, child left_zed_link, origin xyz=0.096 0.0118 0.0407 rpy=0 0 0
- added joint right_zed_joint: type fixed, parent neckPitch_link, child right_zed_link, origin xyz=0.096 -0.0517 0.0407 rpy=0 0 0
