Commit message: add adam_sp

File: adam_inspire/adam_inspire.urdf (robot description, URDF)
Before this commit: robot adam_inspire, 55 links, 54 joints
Links:
- link anklePitchLeft: mass 0.03100000 -> 0.03014230
- link anklePitchRight: mass 0.03100000 -> 0.03014230
- link hipPitchLeft: mass 2.15124786 -> 2.23379987
- link hipPitchRight: mass 2.15124254 -> 2.23477271
- link hipRollLeft: mass 1.29421887 -> 1.35107789
- link hipRollRight: mass 1.29422777 -> 1.35169943
- link pelvis: mass 10.18730021 -> 10.35646604
- link shinLeft: mass 2.19866469 -> 2.25363003
- link shinRight: mass 2.20809154 -> 2.25459286
- link thighLeft: mass 6.64749717 -> 6.43432838
- link thighRight: mass 6.64754534 -> 6.43084152
- link toeLeft: mass 0.47580000 -> 0.63479601
- link toeRight: mass 0.47580000 -> 0.63480789
- link torso: mass 13.28595962 -> 12.89652496
- link waistPitch: mass 0.49870000 -> 0.56353776
- link waistRoll: mass 2.18430742 -> 2.36268465

File: adam_lite/adam_lite.urdf (robot description, URDF)
Before this commit: robot adam_lite, 27 links, 26 joints
Links:
- link anklePitchLeft: mass 0.03100000 -> 0.03014230
- link anklePitchRight: mass 0.03100000 -> 0.03014230
- link hipPitchLeft: mass 2.15124786 -> 2.23379987
- link hipPitchRight: mass 2.15124254 -> 2.23477271
- link hipRollLeft: mass 1.29421887 -> 1.35107789
- link hipRollRight: mass 1.29422777 -> 1.35169943
- link pelvis: mass 10.18730021 -> 10.35646604
- link shinLeft: mass 2.19866469 -> 2.25363003
- link shinRight: mass 2.20809154 -> 2.25459286
- link thighLeft: mass 6.64749717 -> 6.43432838
- link thighRight: mass 6.64754534 -> 6.43084152
- link toeLeft: mass 0.47580000 -> 0.63479601
- link toeRight: mass 0.47580000 -> 0.63480789
- link torso: mass 13.28595962 -> 12.89652496
- link waistPitch: mass 0.49870000 -> 0.56353776
- link waistRoll: mass 2.18430742 -> 2.36268465

File: adam_sp_agx_ir/adam_sp_agx_ir.urdf (robot description, URDF)
Before this commit: robot standard_plus29_agx, 55 links, 54 joints
Links:
- link anklePitchLeft: mass 0.03100000 -> 0.03014230
- link anklePitchRight: mass 0.03100000 -> 0.03014230
- link hipPitchLeft: mass 2.15124786 -> 2.23379987
- link hipPitchRight: mass 2.15124254 -> 2.23477271
- link hipRollLeft: mass 1.29421887 -> 1.35107789
- link hipRollRight: mass 1.29422777 -> 1.35169943
- link pelvis: mass 10.18730021 -> 10.35646604
- link shinLeft: mass 2.19866469 -> 2.25363003
- link shinRight: mass 2.20809154 -> 2.25459286
- link thighLeft: mass 6.64749717 -> 6.43432838
- link thighRight: mass 6.64754534 -> 6.43084152
- link toeLeft: mass 0.47580000 -> 0.63479601
- link toeRight: mass 0.47580000 -> 0.63480789
- link torso: mass 15.33112381 -> 12.89652496
- link waistPitch: mass 0.49870000 -> 0.56353776
- link waistRoll: mass 2.18430742 -> 2.36268465
