Commit message: update meshes path

File: adam_inspire/adam_inspire.urdf (robot description, URDF)
Before this commit: robot adam_inspire, 55 links, 54 joints
Links:
- link L_index_distal: geometry collision mesh filename=meshes/L_index_distal.dae; visual mesh filename=meshes/L_index_distal.dae
- link L_index_proximal: geometry collision mesh filename=meshes/L_index_proximal.dae; visual mesh filename=meshes/L_index_proximal.dae
- link L_middle_distal: geometry collision mesh filename=meshes/L_middle_distal.dae; visual mesh filename=meshes/L_middle_distal.dae
- link L_middle_proximal: geometry collision mesh filename=meshes/L_middle_proximal.dae; visual mesh filename=meshes/L_middle_proximal.dae
- link L_pinky_distal: geometry collision mesh filename=meshes/L_pinky_distal.dae; visual mesh filename=meshes/L_pinky_distal.dae
- link L_pinky_proximal: geometry collision mesh filename=meshes/L_pinky_proximal.dae; visual mesh filename=meshes/L_pinky_proximal.dae
- link L_ring_distal: geometry collision mesh filename=meshes/L_ring_distal.dae; visual mesh filename=meshes/L_ring_distal.dae
- link L_ring_proximal: geometry collision mesh filename=meshes/L_ring_proximal.dae; visual mesh filename=meshes/L_ring_proximal.dae
- link L_thumb_distal: geometry collision mesh filename=meshes/L_thumb_distal.dae; visual mesh filename=meshes/L_thumb_distal.dae
- link L_thumb_intermediate: geometry collision mesh filename=meshes/L_thumb_intermediate.dae; visual mesh filename=meshes/L_thumb_intermediate.dae
- link L_thumb_proximal: geometry collision mesh filename=meshes/L_thumb_proximal.dae; visual mesh filename=meshes/L_thumb_proximal.dae
- link L_thumb_proximal_base: geometry collision mesh filename=meshes/L_thumb_proximal_base.dae; visual mesh filename=meshes/L_thumb_proximal_base.dae
- link R_index_distal: geometry collision mesh filename=meshes/R_index_distal.dae; visual mesh filename=meshes/R_index_distal.dae
- link R_index_distalR_middle_proximal: geometry collision mesh filename=meshes/R_index_distalR_middle_proximal.dae; visual mesh filename=meshes/R_index_distalR_middle_proximal.dae
- link R_index_proximal: geometry collision mesh filename=meshes/R_index_proximal.dae; visual mesh filename=meshes/R_index_proximal.dae
- link R_middle_distal: geometry collision mesh filename=meshes/R_middle_distal.dae; visual mesh filename=meshes/R_middle_distal.dae
- link R_pinky_distal: geometry collision mesh filename=meshes/R_pinky_distal.dae; visual mesh filename=meshes/R_pinky_distal.dae
- link R_pinky_proximal: geometry collision mesh filename=meshes/R_pinky_proximal.dae; visual mesh filename=meshes/R_pinky_proximal.dae
- link R_ring_distal: geometry collision mesh filename=meshes/R_ring_distal.dae; visual mesh filename=meshes/R_ring_distal.dae
- link R_ring_proximal: geometry collision mesh filename=meshes/R_ring_proximal.dae; visual mesh filename=meshes/R_ring_proximal.dae
- link R_thumb_distal: geometry collision mesh filename=meshes/R_thumb_distal.dae; visual mesh filename=meshes/R_thumb_distal.dae
- link R_thumb_intermediate: geometry collision mesh filename=meshes/R_thumb_intermediate.dae; visual mesh filename=meshes/R_thumb_intermediate.dae
- link R_thumb_proximal: geometry collision mesh filename=meshes/R_thumb_proximal.dae; visual mesh filename=meshes/R_thumb_proximal.dae
- link R_thumb_proximal_base: geometry collision mesh filename=meshes/R_thumb_proximal_base.dae; visual mesh filename=meshes/R_thumb_proximal_base.dae
- link anklePitchLeft: geometry visual mesh filename=meshes/anklePitchLeft.dae
- link anklePitchRight: geometry visual mesh filename=meshes/anklePitchRight.dae
- link elbowLeft: geometry visual mesh filename=meshes/elbowLeft.dae
- link elbowRight: geometry visual mesh filename=meshes/elbowRight.dae
- link hipPitchLeft: geometry visual mesh filename=meshes/hipPitchLeft.dae
- link hipPitchRight: geometry visual mesh filename=meshes/hipPitchRight.dae
- link hipRollLeft: geometry visual mesh filename=meshes/hipRollLeft.dae
- link hipRollRight: geometry visual mesh filename=meshes/hipRollRight.dae
- link imu_link: geometry visual mesh filename=meshes/vn100-0001.dae
- link pelvis: geometry collision cylinder length=0.1 radius=0.1; visual mesh filename=meshes/pelvis.dae
- link shinLeft: geometry collision cylinder length=0.22 radius=0.04; visual mesh filename=meshes/shinLeft.dae
- link shinRight: geometry collision cylinder length=0.22 radius=0.04; visual mesh filename=meshes/shinRight.dae
- link shoulderPitchLeft: geometry visual mesh filename=meshes/shoulderPitchLeft.dae
- link shoulderPitchRight: geometry visual mesh filename=meshes/shoulderPitchRight.dae
- link shoulderRollLeft: geometry collision cylinder length=0.02 radius=0.035; visual mesh filename=meshes/shoulderRollLeft.dae
- link shoulderRollRight: geometry collision cylinder length=0.02 radius=0.035; visual mesh filename=meshes/shoulderRollRight.dae
- link shoulderYawLeft: geometry collision cylinder length=0.067 radius=0.0415; visual mesh filename=meshes/shoulderYawLeft.dae
- link shoulderYawRight: geometry collision cylinder length=0.067 radius=0.0415; visual mesh filename=meshes/shoulderYawRight.dae
- link thighLeft: geometry collision cylinder length=0.08 radius=0.06; visual mesh filename=meshes/thighLeft.dae
- link thighRight: geometry collision cylinder length=0.08 radius=0.06; visual mesh filename=meshes/thighRight.dae
- link toeLeft: geometry collision mesh filename=meshes/toeLeft.dae; visual mesh filename=meshes/toeLeft.dae
- link toeRight: geometry collision mesh filename=meshes/toeRight.dae; visual mesh filename=meshes/toeRight.dae
- link torso: geometry collision sphere radius=0.13; visual mesh filename=meshes/torso.dae
- link waistPitch: geometry visual mesh filename=meshes/waistPitch.dae
- link waistRoll: geometry visual mesh filename=meshes/waistRoll.dae
- link wristPitchLeft: geometry visual mesh filename=meshes/wristPitchLeft.dae
- link wristPitchRight: geometry visual mesh filename=meshes/wristPitchRight.dae
- link wristRollLeft: geometry collision mesh filename=meshes/inspire_Left.dae; visual mesh filename=meshes/inspire_Left.dae
- link wristRollRight: geometry collision mesh filename=meshes/inspire_Right.dae; visual mesh filename=meshes/inspire_Right.dae
- link wristYawLeft: geometry collision cylinder length=0.1 radius=0.038; visual mesh filename=meshes/wristYawLeft.dae
- link wristYawRight: geometry collision cylinder length=0.1 radius=0.038; visual mesh filename=meshes/wristYawRight.dae

File: adam_lite/adam_lite.urdf (robot description, URDF)
Before this commit: robot adam_lite, 27 links, 26 joints
Links:
- link anklePitchLeft: geometry visual mesh filename=meshes/anklePitchLeft.dae
- link anklePitchRight: geometry visual mesh filename=meshes/anklePitchRight.dae
- link elbowLeft: geometry visual mesh filename=meshes/elbowLeft.dae
- link elbowRight: geometry visual mesh filename=meshes/elbowRight.dae
- link hipPitchLeft: geometry visual mesh filename=meshes/hipPitchLeft.dae
- link hipPitchRight: geometry visual mesh filename=meshes/hipPitchRight.dae
- link hipRollLeft: geometry visual mesh filename=meshes/hipRollLeft.dae
- link hipRollRight: geometry visual mesh filename=meshes/hipRollRight.dae
- link imu_link: geometry visual mesh filename=meshes/vn100-0001.dae
- link pelvis: geometry collision cylinder length=0.1 radius=0.1; visual mesh filename=meshes/pelvis.dae
- link shinLeft: geometry collision cylinder length=0.22 radius=0.04; visual mesh filename=meshes/shinLeft.dae
- link shinRight: geometry collision cylinder length=0.22 radius=0.04; visual mesh filename=meshes/shinRight.dae
- link shoulderPitchLeft: geometry visual mesh filename=meshes/shoulderPitchLeft.dae
- link shoulderPitchRight: geometry visual mesh filename=meshes/shoulderPitchRight.dae
- link shoulderRollLeft: geometry collision cylinder length=0.02 radius=0.035; visual mesh filename=meshes/shoulderRollLeft.dae
- link shoulderRollRight: geometry collision cylinder length=0.02 radius=0.035; visual mesh filename=meshes/shoulderRollRight.dae
- link shoulderYawLeft: geometry collision cylinder length=0.067 radius=0.0415; visual mesh filename=meshes/shoulderYawLeft.dae
- link shoulderYawRight: geometry collision cylinder length=0.067 radius=0.0415; visual mesh filename=meshes/shoulderYawRight.dae
- link thighLeft: geometry collision cylinder length=0.08 radius=0.06; visual mesh filename=meshes/thighLeft.dae
- link thighRight: geometry collision cylinder length=0.08 radius=0.06; visual mesh filename=meshes/thighRight.dae
- link toeLeft: geometry collision mesh filename=meshes/toeLeft.dae; visual mesh filename=meshes/toeLeft.dae
- link toeRight: geometry collision mesh filename=meshes/toeRight.dae; visual mesh filename=meshes/toeRight.dae
- link torso: geometry collision sphere radius=0.13; visual mesh filename=meshes/torso.dae
- link waistPitch: geometry visual mesh filename=meshes/waistPitch.dae
- link waistRoll: geometry visual mesh filename=meshes/waistRoll.dae
- link wristYawLeft: geometry collision cylinder length=0.25 radius=0.035; visual mesh filename=meshes/wristYawLeft.dae
- link wristYawRight: geometry collision cylinder length=0.25 radius=0.035; visual mesh filename=meshes/wristYawRight.dae

File: adam_sp/adam_sp.urdf (robot description, URDF)
Before this commit: robot standard_plus29_PNDHand, 56 links, 55 joints
Links:
- removed link world
- link L_index_distal: geometry collision mesh filename=meshes/L_index_distal.STL; visual mesh filename=meshes/L_index_distal.STL
- link L_index_proximal: geometry collision mesh filename=meshes/L_index_proximal.STL; visual mesh filename=meshes/L_index_proximal.STL
- link L_middle_distal: geometry collision mesh filename=meshes/L_middle_distal.STL; visual mesh filename=meshes/L_middle_distal.STL
- link L_middle_proximal: geometry collision mesh filename=meshes/L_middle_proximal.STL; visual mesh filename=meshes/L_middle_proximal.STL
- link L_pinky_distal: geometry collision mesh filename=meshes/L_pinky_distal.STL; visual mesh filename=meshes/L_pinky_distal.STL
- link L_pinky_proximal: geometry collision mesh filename=meshes/L_pinky_proximal.STL; visual mesh filename=meshes/L_pinky_proximal.STL
- link L_ring_distal: geometry collision mesh filename=meshes/L_ring_distal.STL; visual mesh filename=meshes/L_ring_distal.STL
- link L_ring_proximal: geometry collision mesh filename=meshes/L_ring_proximal.STL; visual mesh filename=meshes/L_ring_proximal.STL
- link L_thumb_distal: geometry collision mesh filename=meshes/L_thumb_distal.STL; visual mesh filename=meshes/L_thumb_distal.STL
- link L_thumb_intermediate: geometry collision mesh filename=meshes/L_thumb_intermediate.STL; visual mesh filename=meshes/L_thumb_intermediate.STL
- link L_thumb_proximal: geometry collision mesh filename=meshes/L_thumb_proximal.STL; visual mesh filename=meshes/L_thumb_proximal.STL
- link L_thumb_proximal_base: geometry collision mesh filename=meshes/L_thumb_proximal_base.STL; visual mesh filename=meshes/L_thumb_proximal_base.STL
- link R_index_distal: geometry collision mesh filename=meshes/R_index_distal.STL; visual mesh filename=meshes/R_index_distal.STL
- link R_index_proximal: geometry collision mesh filename=meshes/R_index_proximal.STL; visual mesh filename=meshes/R_index_proximal.STL
- link R_middle_distal: geometry collision mesh filename=meshes/R_middle_distal.STL; visual mesh filename=meshes/R_middle_distal.STL
- link R_middle_proximal: geometry collision mesh filename=meshes/R_middle_proximal.STL; visual mesh filename=meshes/R_middle_proximal.STL
- link R_pinky_distal: geometry collision mesh filename=meshes/R_pinky_distal.STL; visual mesh filename=meshes/R_pinky_distal.STL
- link R_pinky_proximal: geometry collision mesh filename=meshes/R_pinky_proximal.STL; visual mesh filename=meshes/R_pinky_proximal.STL
- link R_ring_distal: geometry collision mesh filename=meshes/R_ring_distal.STL; visual mesh filename=meshes/R_ring_distal.STL
- link R_ring_proximal: geometry collision mesh filename=meshes/R_ring_proximal.STL; visual mesh filename=meshes/R_ring_proximal.STL
- link R_thumb_distal: geometry collision mesh filename=meshes/R_thumb_distal.STL; visual mesh filename=meshes/R_thumb_distal.STL
- link R_thumb_intermediate: geometry collision mesh filename=meshes/R_thumb_intermediate.STL; visual mesh filename=meshes/R_thumb_intermediate.STL
- link R_thumb_proximal: geometry collision mesh filename=meshes/R_thumb_proximal.STL; visual mesh filename=meshes/R_thumb_proximal.STL
- link R_thumb_proximal_base: geometry collision mesh filename=meshes/R_thumb_proximal_base.STL; visual mesh filename=meshes/R_thumb_proximal_base.STL
- link anklePitchLeft: geometry visual mesh filename=meshes/anklePitchLeft.dae
- link anklePitchRight: geometry visual mesh filename=meshes/anklePitchRight.dae
- link elbowLeft: geometry visual mesh filename=meshes/elbowLeft.dae
- link elbowRight: geometry visual mesh filename=meshes/elbowRight.dae
- link hipPitchLeft: geometry visual mesh filename=meshes/hipPitchLeft.dae
- link hipPitchRight: geometry visual mesh filename=meshes/hipPitchRight.dae
- link hipRollLeft: geometry visual mesh filename=meshes/hipRollLeft.dae
- link hipRollRight: geometry visual mesh filename=meshes/hipRollRight.dae
- link imu_link: geometry visual mesh filename=meshes/vn100-0001.dae
- link pelvis: geometry collision cylinder length=0.1 radius=0.1; visual mesh filename=meshes/pelvis.dae
- link shinLeft: geometry collision cylinder length=0.22 radius=0.04; visual mesh filename=meshes/shinLeft.dae
- link shinRight: geometry collision cylinder length=0.22 radius=0.04; visual mesh filename=meshes/shinRight.dae
- link shoulderPitchLeft: geometry visual mesh filename=meshes/shoulderPitchLeft.dae
- link shoulderPitchRight: geometry visual mesh filename=meshes/shoulderPitchRight.dae
- link shoulderRollLeft: geometry collision cylinder length=0.02 radius=0.035; visual mesh filename=meshes/shoulderRollLeft.dae
- link shoulderRollRight: geometry collision cylinder length=0.02 radius=0.035; visual mesh filename=meshes/shoulderRollRight.dae
- link shoulderYawLeft: geometry collision cylinder length=0.067 radius=0.0415; visual mesh filename=meshes/shoulderYawLeft.dae
- link shoulderYawRight: geometry collision cylinder length=0.067 radius=0.0415; visual mesh filename=meshes/shoulderYawRight.dae
- link thighLeft: geometry collision cylinder length=0.08 radius=0.06; visual mesh filename=meshes/thighLeft.dae
- link thighRight: geometry collision cylinder length=0.08 radius=0.06; visual mesh filename=meshes/thighRight.dae
- link toeLeft: geometry collision mesh filename=meshes/toeLeft.dae; visual mesh filename=meshes/toeLeft.dae
- link toeRight: geometry collision mesh filename=meshes/toeRight.dae; visual mesh filename=meshes/toeRight.dae
- link torso: geometry collision sphere radius=0.13; visual mesh filename=meshes/torso.dae
- link waistPitch: geometry visual mesh filename=meshes/waistPitch.dae
- link waistRoll: geometry visual mesh filename=meshes/waistRoll.dae
- link wristPitchLeft: geometry visual mesh filename=meshes/wristPitchLeft.dae
- link wristPitchRight: geometry visual mesh filename=meshes/wristPitchRight.dae
- link wristRollLeft: geometry collision mesh filename=meshes/wristRollLeft.STL; visual mesh filename=meshes/wristRollLeft.STL
- link wristRollRight: geometry collision mesh filename=meshes/wristRollRight.STL; visual mesh filename=meshes/wristRollRight.STL
- link wristYawLeft: geometry collision cylinder length=0.1 radius=0.038; visual mesh filename=meshes/wristYawLeft.dae
- link wristYawRight: geometry collision cylinder length=0.1 radius=0.038; visual mesh filename=meshes/wristYawRight.dae
Joints:
- removed joint floating_joint

File: adam_sp_agx_ir/adam_sp_agx_ir.urdf (robot description, URDF)
Before this commit: robot standard_plus29_agx, 55 links, 54 joints
Links:
- link L_index_distal: geometry collision mesh filename=meshes/L_index_distal.dae; visual mesh filename=meshes/L_index_distal.dae
- link L_index_proximal: geometry collision mesh filename=meshes/L_index_proximal.dae; visual mesh filename=meshes/L_index_proximal.dae
- link L_middle_distal: geometry collision mesh filename=meshes/L_middle_distal.dae; visual mesh filename=meshes/L_middle_distal.dae
- link L_middle_proximal: geometry collision mesh filename=meshes/L_middle_proximal.dae; visual mesh filename=meshes/L_middle_proximal.dae
- link L_pinky_distal: geometry collision mesh filename=meshes/L_pinky_distal.dae; visual mesh filename=meshes/L_pinky_distal.dae
- link L_pinky_proximal: geometry collision mesh filename=meshes/L_pinky_proximal.dae; visual mesh filename=meshes/L_pinky_proximal.dae
- link L_ring_distal: geometry collision mesh filename=meshes/L_ring_distal.dae; visual mesh filename=meshes/L_ring_distal.dae
- link L_ring_proximal: geometry collision mesh filename=meshes/L_ring_proximal.dae; visual mesh filename=meshes/L_ring_proximal.dae
- link L_thumb_distal: geometry collision mesh filename=meshes/L_thumb_distal.dae; visual mesh filename=meshes/L_thumb_distal.dae
- link L_thumb_intermediate: geometry collision mesh filename=meshes/L_thumb_intermediate.dae; visual mesh filename=meshes/L_thumb_intermediate.dae
- link L_thumb_proximal: geometry collision mesh filename=meshes/L_thumb_proximal.dae; visual mesh filename=meshes/L_thumb_proximal.dae
- link L_thumb_proximal_base: geometry collision mesh filename=meshes/L_thumb_proximal_base.dae; visual mesh filename=meshes/L_thumb_proximal_base.dae
- link R_index_distal: geometry collision mesh filename=meshes/R_index_distal.dae; visual mesh filename=meshes/R_index_distal.dae
- link R_index_distalR_middle_proximal: geometry collision mesh filename=meshes/R_index_distalR_middle_proximal.dae; visual mesh filename=meshes/R_index_distalR_middle_proximal.dae
- link R_index_proximal: geometry collision mesh filename=meshes/R_index_proximal.dae; visual mesh filename=meshes/R_index_proximal.dae
- link R_middle_distal: geometry collision mesh filename=meshes/R_middle_distal.dae; visual mesh filename=meshes/R_middle_distal.dae
- link R_pinky_distal: geometry collision mesh filename=meshes/R_pinky_distal.dae; visual mesh filename=meshes/R_pinky_distal.dae
- link R_pinky_proximal: geometry collision mesh filename=meshes/R_pinky_proximal.dae; visual mesh filename=meshes/R_pinky_proximal.dae
- link R_ring_distal: geometry collision mesh filename=meshes/R_ring_distal.dae; visual mesh filename=meshes/R_ring_distal.dae
- link R_ring_proximal: geometry collision mesh filename=meshes/R_ring_proximal.dae; visual mesh filename=meshes/R_ring_proximal.dae
- link R_thumb_distal: geometry collision mesh filename=meshes/R_thumb_distal.dae; visual mesh filename=meshes/R_thumb_distal.dae
- link R_thumb_intermediate: geometry collision mesh filename=meshes/R_thumb_intermediate.dae; visual mesh filename=meshes/R_thumb_intermediate.dae
- link R_thumb_proximal: geometry collision mesh filename=meshes/R_thumb_proximal.dae; visual mesh filename=meshes/R_thumb_proximal.dae
- link R_thumb_proximal_base: geometry collision mesh filename=meshes/R_thumb_proximal_base.dae; visual mesh filename=meshes/R_thumb_proximal_base.dae
- link anklePitchLeft: geometry visual mesh filename=meshes/anklePitchLeft.dae
- link anklePitchRight: geometry visual mesh filename=meshes/anklePitchRight.dae
- link elbowLeft: geometry visual mesh filename=meshes/elbowLeft.dae
- link elbowRight: geometry visual mesh filename=meshes/elbowRight.dae
- link hipPitchLeft: geometry visual mesh filename=meshes/hipPitchLeft.dae
- link hipPitchRight: geometry visual mesh filename=meshes/hipPitchRight.dae
- link hipRollLeft: geometry visual mesh filename=meshes/hipRollLeft.dae
- link hipRollRight: geometry visual mesh filename=meshes/hipRollRight.dae
- link imu_link: geometry visual mesh filename=meshes/vn100-0001.dae
- link pelvis: geometry collision cylinder length=0.1 radius=0.1; visual mesh filename=meshes/pelvis.dae
- link shinLeft: geometry collision cylinder length=0.22 radius=0.04; visual mesh filename=meshes/shinLeft.dae
- link shinRight: geometry collision cylinder length=0.22 radius=0.04; visual mesh filename=meshes/shinRight.dae
- link shoulderPitchLeft: geometry visual mesh filename=meshes/shoulderPitchLeft.dae
- link shoulderPitchRight: geometry visual mesh filename=meshes/shoulderPitchRight.dae
- link shoulderRollLeft: geometry collision cylinder length=0.02 radius=0.035; visual mesh filename=meshes/shoulderRollLeft.dae
- link shoulderRollRight: geometry collision cylinder length=0.02 radius=0.035; visual mesh filename=meshes/shoulderRollRight.dae
- link shoulderYawLeft: geometry collision cylinder length=0.067 radius=0.0415; visual mesh filename=meshes/shoulderYawLeft.dae
- link shoulderYawRight: geometry collision cylinder length=0.067 radius=0.0415; visual mesh filename=meshes/shoulderYawRight.dae
- link thighLeft: geometry collision cylinder length=0.08 radius=0.06; visual mesh filename=meshes/thighLeft.dae
- link thighRight: geometry collision cylinder length=0.08 radius=0.06; visual mesh filename=meshes/thighRight.dae
- link toeLeft: geometry collision mesh filename=meshes/toeLeft.dae; visual mesh filename=meshes/toeLeft.dae
- link toeRight: geometry collision mesh filename=meshes/toeRight.dae; visual mesh filename=meshes/toeRight.dae
- link torso: geometry collision sphere radius=0.13; visual mesh filename=meshes/torso.dae
- link waistPitch: geometry visual mesh filename=meshes/waistPitch.dae
- link waistRoll: geometry visual mesh filename=meshes/waistRoll.dae
- link wristPitchLeft: geometry visual mesh filename=meshes/wristPitchLeft.dae
- link wristPitchRight: geometry visual mesh filename=meshes/wristPitchRight.dae
- link wristRollLeft: geometry collision mesh filename=meshes/inspire_Left.dae; visual mesh filename=meshes/inspire_Left.dae
- link wristRollRight: geometry collision mesh filename=meshes/inspire_Right.dae; visual mesh filename=meshes/inspire_Right.dae
- link wristYawLeft: geometry collision cylinder length=0.1 radius=0.038; visual mesh filename=meshes/wristYawLeft.dae
- link wristYawRight: geometry collision cylinder length=0.1 radius=0.038; visual mesh filename=meshes/wristYawRight.dae
