Commit message: Update mesh filenames and add new COLLADA files for adam variants

File: adam_inspire/adam_inspire.urdf (robot description, URDF)
Before this commit: robot adam_inspire, 55 links, 54 joints
Links:
- link imu_link: geometry visual mesh filename=meshes/vn100_0001.dae

File: adam_lite/adam_lite.urdf (robot description, URDF)
Before this commit: robot adam_lite, 27 links, 26 joints
Links:
- link imu_link: geometry visual mesh filename=meshes/vn100_0001.dae

File: adam_lite_agx/adam_lite_agx.urdf (robot description, URDF)
Before this commit: robot adam_lite_agx, 27 links, 26 joints
Links:
- link imu_link: geometry visual mesh filename=meshes/vn100_0001.dae

File: adam_sp/adam_sp.urdf (robot description, URDF)
Before this commit: robot adam_sp, 55 links, 54 joints
Links:
- link imu_link: geometry visual mesh filename=meshes/vn100_0001.dae

File: adam_sp_agx_ir/adam_sp_agx_ir.urdf (robot description, URDF)
Before this commit: robot standard_plus29_agx, 55 links, 54 joints
Links:
- link imu_link: geometry visual mesh filename=meshes/vn100_0001.dae

File: adam_standard/adam_standard.urdf (robot description, URDF)
Before this commit: robot adam_standard, 29 links, 28 joints
Links:
- link imu_link: geometry visual mesh filename=meshes/vn100_0001.dae
