Commit message: debug omnipicker

File: adam_pro_omnipicker/adam_pro_omnipicker.urdf (robot description, URDF)
Before this commit: robot adam_pro_omnipicker, 57 links, 56 joints
Joints:
- removed joint op_l_hand_narrow1_joint
- removed joint op_r_hand_narrow1_joint
- added joint left_gripper_joint: type revolute, parent op_l_base_link, child op_l_hand_narrow1_Link, origin xyz=0 -0.0195 0.0565 rpy=-2.9951 -1.5708 -0.15964, axis 0 0 1, limit lower=0.01 upper=0.78 effort=50 velocity=3.141592653589793
- added joint right_gripper_joint: type revolute, parent op_r_base_link, child op_r_hand_narrow1_Link, origin xyz=0 -0.0195 0.0565 rpy=-2.9951 -1.5708 -0.15964, axis 0 0 1, limit lower=0.01 upper=0.785 effort=50 velocity=3.141592653589793
- joint op_l_hand_narrow2_joint: limit lower=-3.14 upper=3.14 effort=0 velocity=0 -> lower=-3.141592653589793 upper=3.141592653589793 effort=50 velocity=3.141592653589793; mimic (none) -> joint=left_gripper_joint multiplier=0.02 offset=0
- joint op_l_hand_narrow3_joint: limit lower=-3.14 upper=3.14 effort=0 velocity=0 -> lower=-3.141592653589793 upper=3.141592653589793 effort=50 velocity=3.141592653589793; mimic (none) -> joint=left_gripper_joint multiplier=0.4 offset=0
- joint op_l_hand_narrow4_joint: limit lower=-3.14 upper=3.14 effort=0 velocity=0 -> lower=-3.141592653589793 upper=3.141592653589793 effort=50 velocity=3.141592653589793
- joint op_l_hand_narrow_loop_joint: axis 0 0 -1 -> 0 0 1; limit lower=-3.14 upper=3.14 effort=0 velocity=0 -> lower=-3.141592653589793 upper=3.141592653589793 effort=50 velocity=3.141592653589793; mimic (none) -> joint=left_gripper_joint multiplier=1.5 offset=0
- joint op_l_hand_wide1_joint: limit lower=-3.14 upper=3.14 effort=0 velocity=0 -> lower=-3.141592653589793 upper=3.141592653589793 effort=50 velocity=3.141592653589793; mimic (none) -> joint=left_gripper_joint multiplier=1 offset=0
- joint op_l_hand_wide2_joint: axis 0 0 -1 -> 0 0 1; limit lower=-3.14 upper=3.14 effort=0 velocity=0 -> lower=-3.141592653589793 upper=3.141592653589793 effort=50 velocity=3.141592653589793; mimic (none) -> joint=left_gripper_joint multiplier=0.02 offset=0
- joint op_l_hand_wide3_joint: axis 0 0 -1 -> 0 0 1; limit lower=-3.14 upper=3.14 effort=0 velocity=0 -> lower=-3.141592653589793 upper=3.141592653589793 effort=50 velocity=3.141592653589793; mimic (none) -> joint=left_gripper_joint multiplier=0.4 offset=0
- joint op_l_hand_wide4_joint: limit lower=-3.14 upper=3.14 effort=0 velocity=0 -> (none)
- joint op_l_hand_wide_loop_joint: limit lower=-3.14 upper=3.14 effort=0 velocity=0 -> lower=-3.141592653589793 upper=3.141592653589793 effort=50 velocity=3.141592653589793; mimic (none) -> joint=left_gripper_joint multiplier=1.5 offset=0
- joint op_r_hand_narrow2_joint: limit lower=-3.14 upper=3.14 effort=0 velocity=0 -> lower=-3.141592653589793 upper=3.141592653589793 effort=50 velocity=3.141592653589793; mimic (none) -> joint=right_gripper_joint multiplier=0.02 offset=0
- joint op_r_hand_narrow3_joint: limit lower=-3.14 upper=3.14 effort=0 velocity=0 -> lower=-3.141592653589793 upper=3.141592653589793 effort=50 velocity=3.141592653589793; mimic (none) -> joint=right_gripper_joint multiplier=0.4 offset=0
- joint op_r_hand_narrow_loop_joint: axis 0 0 -1 -> 0 0 1; limit lower=-3.14 upper=3.14 effort=0 velocity=0 -> lower=-3.141592653589793 upper=3.141592653589793 effort=50 velocity=3.141592653589793; mimic (none) -> joint=right_gripper_joint multiplier=1.5 offset=0
- joint op_r_hand_wide1_joint: limit lower=-3.14 upper=3.14 effort=0 velocity=0 -> lower=-3.141592653589793 upper=3.141592653589793 effort=50 velocity=3.141592653589793; mimic (none) -> joint=right_gripper_joint multiplier=1 offset=0
- joint op_r_hand_wide2_joint: axis 0 0 -1 -> 0 0 1; limit lower=-3.14 upper=3.14 effort=0 velocity=0 -> lower=-3.141592653589793 upper=3.141592653589793 effort=50 velocity=3.141592653589793; mimic (none) -> joint=right_gripper_joint multiplier=0.02 offset=0
- joint op_r_hand_wide3_joint: axis 0 0 -1 -> 0 0 1; limit lower=-3.14 upper=3.14 effort=0 velocity=0 -> lower=-3.141592653589793 upper=3.141592653589793 effort=50 velocity=3.141592653589793; mimic (none) -> joint=right_gripper_joint multiplier=0.4 offset=0
- joint op_r_hand_wide_loop_joint: limit lower=-3.14 upper=3.14 effort=0 velocity=0 -> lower=-3.141592653589793 upper=3.141592653589793 effort=50 velocity=3.141592653589793; mimic (none) -> joint=right_gripper_joint multiplier=1.5 offset=0

File: adam_u_omnipicker/adam_u_omnipicker.urdf (robot description, URDF)
Before this commit: robot adam_u_omnipicker, 42 links, 41 joints
Links:
- added link left_zed_link
- added link right_zed_link
Joints:
- removed joint op_l_hand_narrow1_joint
- removed joint op_r_hand_narrow1_joint
- added joint left_gripper_joint: type revolute, parent op_l_base_link, child op_l_hand_narrow1_Link, origin xyz=0 -0.0195 0.0565 rpy=-2.9951 -1.5708 -0.15964, axis 0 0 1, limit lower=0.01 upper=0.78 effort=50 velocity=3.141592653589793
- added joint left_zed_joint: type fixed, parent neckPitch_link, child left_zed_link, origin xyz=0.096 0.0118 0.0407 rpy=0 0 0
- added joint right_gripper_joint: type revolute, parent op_r_base_link, child op_r_hand_narrow1_Link, origin xyz=0 -0.0195 0.0565 rpy=-2.9951 -1.5708 -0.15964, axis 0 0 1, limit lower=0.01 upper=0.785 effort=50 velocity=3.141592653589793
- added joint right_zed_joint: type fixed, parent neckPitch_link, child right_zed_link, origin xyz=0.096 -0.0517 0.0407 rpy=0 0 0
- joint op_l_hand_narrow2_joint: limit lower=-3.14 upper=3.14 effort=0 velocity=0 -> lower=-3.141592653589793 upper=3.141592653589793 effort=50 velocity=3.141592653589793; mimic (none) -> joint=left_gripper_joint multiplier=0.02 offset=0
- joint op_l_hand_narrow3_joint: limit lower=-3.14 upper=3.14 effort=0 velocity=0 -> lower=-3.141592653589793 upper=3.141592653589793 effort=50 velocity=3.141592653589793; mimic (none) -> joint=left_gripper_joint multiplier=0.4 offset=0
- joint op_l_hand_narrow4_joint: limit lower=-3.14 upper=3.14 effort=0 velocity=0 -> lower=-3.141592653589793 upper=3.141592653589793 effort=50 velocity=3.141592653589793
- joint op_l_hand_narrow_loop_joint: axis 0 0 -1 -> 0 0 1; limit lower=-3.14 upper=3.14 effort=0 velocity=0 -> lower=-3.141592653589793 upper=3.141592653589793 effort=50 velocity=3.141592653589793; mimic (none) -> joint=left_gripper_joint multiplier=1.5 offset=0
- joint op_l_hand_wide1_joint: limit lower=-3.14 upper=3.14 effort=0 velocity=0 -> lower=-3.141592653589793 upper=3.141592653589793 effort=50 velocity=3.141592653589793; mimic (none) -> joint=left_gripper_joint multiplier=1 offset=0
- joint op_l_hand_wide2_joint: axis 0 0 -1 -> 0 0 1; limit lower=-3.14 upper=3.14 effort=0 velocity=0 -> lower=-3.141592653589793 upper=3.141592653589793 effort=50 velocity=3.141592653589793; mimic (none) -> joint=left_gripper_joint multiplier=0.02 offset=0
- joint op_l_hand_wide3_joint: axis 0 0 -1 -> 0 0 1; limit lower=-3.14 upper=3.14 effort=0 velocity=0 -> lower=-3.141592653589793 upper=3.141592653589793 effort=50 velocity=3.141592653589793; mimic (none) -> joint=left_gripper_joint multiplier=0.4 offset=0
- joint op_l_hand_wide4_joint: limit lower=-3.14 upper=3.14 effort=0 velocity=0 -> (none)
- joint op_l_hand_wide_loop_joint: limit lower=-3.14 upper=3.14 effort=0 velocity=0 -> lower=-3.141592653589793 upper=3.141592653589793 effort=50 velocity=3.141592653589793; mimic (none) -> joint=left_gripper_joint multiplier=1.5 offset=0
- joint op_r_hand_narrow2_joint: limit lower=-3.14 upper=3.14 effort=0 velocity=0 -> lower=-3.141592653589793 upper=3.141592653589793 effort=50 velocity=3.141592653589793; mimic (none) -> joint=right_gripper_joint multiplier=0.02 offset=0
- joint op_r_hand_narrow3_joint: limit lower=-3.14 upper=3.14 effort=0 velocity=0 -> lower=-3.141592653589793 upper=3.141592653589793 effort=50 velocity=3.141592653589793; mimic (none) -> joint=right_gripper_joint multiplier=0.4 offset=0
- joint op_r_hand_narrow_loop_joint: axis 0 0 -1 -> 0 0 1; limit lower=-3.14 upper=3.14 effort=0 velocity=0 -> lower=-3.141592653589793 upper=3.141592653589793 effort=50 velocity=3.141592653589793; mimic (none) -> joint=right_gripper_joint multiplier=1.5 offset=0
- joint op_r_hand_wide1_joint: limit lower=-3.14 upper=3.14 effort=0 velocity=0 -> lower=-3.141592653589793 upper=3.141592653589793 effort=50 velocity=3.141592653589793; mimic (none) -> joint=right_gripper_joint multiplier=1 offset=0
- joint op_r_hand_wide2_joint: axis 0 0 -1 -> 0 0 1; limit lower=-3.14 upper=3.14 effort=0 velocity=0 -> lower=-3.141592653589793 upper=3.141592653589793 effort=50 velocity=3.141592653589793; mimic (none) -> joint=right_gripper_joint multiplier=0.02 offset=0
- joint op_r_hand_wide3_joint: axis 0 0 -1 -> 0 0 1; limit lower=-3.14 upper=3.14 effort=0 velocity=0 -> lower=-3.141592653589793 upper=3.141592653589793 effort=50 velocity=3.141592653589793; mimic (none) -> joint=right_gripper_joint multiplier=0.4 offset=0
- joint op_r_hand_wide_loop_joint: limit lower=-3.14 upper=3.14 effort=0 velocity=0 -> lower=-3.141592653589793 upper=3.141592653589793 effort=50 velocity=3.141592653589793; mimic (none) -> joint=right_gripper_joint multiplier=1.5 offset=0
